File: f3.sch (KiCad schematic (older format))
At the start: 13 parts, among them U4 STM32F303K8Tx, Y1 Crystal

Commit message: Added I2C level shifter
Connections:
- net labels added: TOF_EN
- net labels removed: 2V8_EN
Changed lines of the file:
@@
 $Descr A4 11693 8268
 encoding utf-8
-Sheet 3 3
+Sheet 3 4
 Title ""
 Date ""
@@
 NoConn ~ 4750 4100
 Text HLabel 6000 3900 2    50   Output ~ 0
-2V8_EN
+TOF_EN
 NoConn ~ 4750 4200
 NoConn ~ 4750 4300

Commit message: Added ToF connectors and fixed schematic ERC
Parts:
- renumbered C9 to C10, C10 to C11, C11 to C12, C12 to C13, C6 to C7, C7 to C8, C8 to C9, D5 to D6, R7 to R8, R8 to R9, U4 to U5
Changed lines of the file:
@@
 $EndDescr
 $Comp
-L MCU_ST_STM32F3:STM32F303K8Tx U4
+L MCU_ST_STM32F3:STM32F303K8Tx U5
 U 1 1 5BBD3F5D
 P 5350 3800
-F 0 "U4" H 5800 2800 50  0000 C CNN
+F 0 "U5" H 5800 2800 50  0000 C CNN
 F 1 "STM32F303K8Tx" H 5800 2700 50  0000 C CNN
 F 2 "Package_QFP:LQFP-32_7x7mm_P0.8mm" H 4850 2900 50  0001 R CNN
@@
 $EndComp
 $Comp
-L Device:C C6
+L Device:C C7
 U 1 1 5BBD416E
 P 3800 3500
-F 0 "C6" V 3548 3500 50  0000 C CNN
+F 0 "C7" V 3548 3500 50  0000 C CNN
 F 1 "C" V 3639 3500 50  0000 C CNN
 F 2 "" H 3838 3350 50  0001 C CNN
@@
 $EndComp
 $Comp
-L Device:C C7
+L Device:C C8
 U 1 1 5BBD4205
 P 3800 4000
-F 0 "C7" V 3548 4000 50  0000 C CNN
+F 0 "C8" V 3548 4000 50  0000 C CNN
 F 1 "C" V 3639 4000 50  0000 C CNN
 F 2 "" H 3838 3850 50  0001 C CNN
@@
 $EndComp
 $Comp
-L power:GND #PWR0115
+L power:GND #PWR040
 U 1 1 5BBD4293
 P 3500 3500
-F 0 "#PWR0115" H 3500 3250 50  0001 C CNN
+F 0 "#PWR040" H 3500 3250 50  0001 C CNN
 F 1 "GND" V 3505 3372 50  0000 R CNN
 F 2 "" H 3500 3500 50  0001 C CNN
@@
 $EndComp
 $Comp
-L power:GND #PWR0116
+L power:GND #PWR041
 U 1 1 5BBD42C5
 P 3500 4000
-F 0 "#PWR0116" H 3500 3750 50  0001 C CNN
+F 0 "#PWR041" H 3500 3750 50  0001 C CNN
 F 1 "GND" V 3505 3872 50  0000 R CNN
 F 2 "" H 3500 4000 50  0001 C CNN
@@
 	4100 3950 4100 3900
 $Comp
-L Device:R R7
+L Device:R R8
 U 1 1 5BBD441A
 P 4400 3300
-F 0 "R7" V 4193 3300 50  0000 C CNN
+F 0 "R8" V 4193 3300 50  0000 C CNN
 F 1 "R" V 4284 3300 50  0000 C CNN
 F 2 "" V 4330 3300 50  0001 C CNN
@@
 	4550 3300 4750 3300
 $Comp
-L power:GND #PWR0117
+L power:GND #PWR039
 U 1 1 5BBD4A9A
 P 3150 3000
-F 0 "#PWR0117" H 3150 2750 50  0001 C CNN
+F 0 "#PWR039" H 3150 2750 50  0001 C CNN
 F 1 "GND" V 3155 2872 50  0000 R CNN
 F 2 "" H 3150 3000 50  0001 C CNN
@@
 	3150 3000 3300 3000
 $Comp
-L power:+3V3 #PWR0118
+L power:+3V3 #PWR043
 U 1 1 5BBD4C69
 P 3900 3000
-F 0 "#PWR0118" H 3900 2850 50  0001 C CNN
+F 0 "#PWR043" H 3900 2850 50  0001 C CNN
 F 1 "+3V3" V 3915 3128 50  0000 L CNN
 F 2 "" H 3900 3000 50  0001 C CNN
@@
 NRST
 $Comp
-L Device:C C8
+L Device:C C9
 U 1 1 5BBD5511
 P 4650 2800
-F 0 "C8" H 4765 2846 50  0000 L CNN
+F 0 "C9" H 4765 2846 50  0000 L CNN
 F 1 "C" H 4765 2755 50  0000 L CNN
 F 2 "" H 4688 2650 50  0001 C CNN
@@
 $EndComp
 $Comp
-L power:GND #PWR0119
+L power:GND #PWR044
 U 1 1 5BBD55CA
 P 4650 2500
-F 0 "#PWR0119" H 4650 2250 50  0001 C CNN
+F 0 "#PWR044" H 4650 2250 50  0001 C CNN
 F 1 "GND" H 4655 2327 50  0000 C CNN
 F 2 "" H 4650 2500 50  0001 C CNN
@@
 	5350 2650 5450 2650
 $Comp
-L power:+3V3 #PWR0120
+L power:+3V3 #PWR049
 U 1 1 5BBD6204
 P 5600 2650
-F 0 "#PWR0120" H 5600 2500 50  0001 C CNN
+F 0 "#PWR049" H 5600 2500 50  0001 C CNN
 F 1 "+3V3" V 5615 2778 50  0000 L CNN
 F 2 "" H 5600 2650 50  0001 C CNN
@@
 Connection ~ 5450 2650
 $Comp
-L Device:C C9
+L Device:C C10
 U 1 1 5BBD657B
 P 5050 2300
-F 0 "C9" V 4798 2300 50  0000 C CNN
+F 0 "C10" V 4798 2300 50  0000 C CNN
 F 1 "C" V 4889 2300 50  0000 C CNN
 F 2 "" H 5088 2150 50  0001 C CNN
@@
 $EndComp
 $Comp
-L Device:C C10
+L Device:C C11
 U 1 1 5BBD660C
 P 5300 2300
-F 0 "C10" H 5185 2346 50  0000 R CNN
+F 0 "C11" H 5185 2346 50  0000 R CNN
 F 1 "C" H 5185 2255 50  0000 R CNN
 F 2 "" H 5338 2150 50  0001 C CNN
@@
 $EndComp
 $Comp
-L Device:C C11
+L Device:C C12
 U 1 1 5BBD669F
 P 5550 2300
-F 0 "C11" V 5298 2300 50  0000 C CNN
+F 0 "C12" V 5298 2300 50  0000 C CNN
 F 1 "C" V 5389 2300 50  0000 C CNN
 F 2 "" H 5588 2150 50  0001 C CNN
@@
 $EndComp
 $Comp
-L Device:C C12
+L Device:C C13
 U 1 1 5BBD681C
 P 5800 2300
-F 0 "C12" V 5548 2300 50  0000 C CNN
+F 0 "C13" V 5548 2300 50  0000 C CNN
 F 1 "C" V 5639 2300 50  0000 C CNN
 F 2 "" H 5838 2150 50  0001 C CNN
@@
 $EndComp
 $Comp
-L power:GND #PWR0121
+L power:GND #PWR050
 U 1 1 5BBD68AE
 P 5800 2050
-F 0 "#PWR0121" H 5800 1800 50  0001 C CNN
+F 0 "#PWR050" H 5800 1800 50  0001 C CNN
 F 1 "GND" V 5805 1922 50  0000 R CNN
 F 2 "" H 5800 2050 50  0001 C CNN
@@
 $EndComp
 $Comp
-L power:GND #PWR0122
+L power:GND #PWR048
 U 1 1 5BBD68FC
 P 5550 2050
-F 0 "#PWR0122" H 5550 1800 50  0001 C CNN
+F 0 "#PWR048" H 5550 1800 50  0001 C CNN
 F 1 "GND" V 5555 1922 50  0000 R CNN
 F 2 "" H 5550 2050 50  0001 C CNN
@@
 $EndComp
 $Comp
-L power:GND #PWR0123
+L power:GND #PWR046
 U 1 1 5BBD694A
 P 5300 2050
-F 0 "#PWR0123" H 5300 1800 50  0001 C CNN
+F 0 "#PWR046" H 5300 1800 50  0001 C CNN
 F 1 "GND" V 5305 1922 50  0000 R CNN
 F 2 "" H 5300 2050 50  0001 C CNN
@@
 $EndComp
 $Comp
-L power:GND #PWR0124
+L power:GND #PWR045
 U 1 1 5BBD6998
 P 5050 2050
-F 0 "#PWR0124" H 5050 1800 50  0001 C CNN
+F 0 "#PWR045" H 5050 1800 50  0001 C CNN
 F 1 "GND" V 5055 1922 50  0000 R CNN
 F 2 "" H 5050 2050 50  0001 C CNN
@@
 	5550 2550 5550 2650
 $Comp
-L power:GND #PWR0125
+L power:GND #PWR047
 U 1 1 5BBDA4B0
 P 5300 4900
-F 0 "#PWR0125" H 5300 4650 50  0001 C CNN
+F 0 "#PWR047" H 5300 4650 50  0001 C CNN
 F 1 "GND" H 5305 4727 50  0000 C CNN
 F 2 "" H 5300 4900 50  0001 C CNN
@@
 Connection ~ 5300 4900
 $Comp
-L Device:R R8
+L Device:R R9
 U 1 1 5BBDC2CE
 P 4450 4500
-F 0 "R8" V 4243 4500 50  0000 C CNN
+F 0 "R9" V 4243 4500 50  0000 C CNN
 F 1 "R" V 4334 4500 50  0000 C CNN
 F 2 "" V 4380 4500 50  0001 C CNN
@@
 $EndComp
 $Comp
-L power:GND #PWR0126
+L power:GND #PWR042
 U 1 1 5BBDC410
 P 3700 4500
-F 0 "#PWR0126" H 3700 4250 50  0001 C CNN
+F 0 "#PWR042" H 3700 4250 50  0001 C CNN
 F 1 "GND" V 3705 4372 50  0000 R CNN
 F 2 "" H 3700 4500 50  0001 C CNN
@@
 $EndComp
 $Comp
-L Device:LED_ALT D5
+L Device:LED_ALT D6
 U 1 1 5BBDC4BF
 P 4000 4500
-F 0 "D5" H 3991 4716 50  0000 C CNN
+F 0 "D6" H 3991 4716 50  0000 C CNN
 F 1 "LED_ALT" H 3991 4625 50  0000 C CNN
 F 2 "" H 4000 4500 50  0001 C CNN

Commit message: Update F3 for ultrasonic sensors and shift register
Connections:
- net labels added: TOF_RESET_DATA, TOF_RESET_SHIFT, US_ECHO_0, US_ECHO_1, US_ECHO_2, US_ECHO_3, US_TRIG_0, US_TRIG_1, US_TRIG_2, US_TRIG_3
- net labels removed: TOF_EN, ToF_Reset_0, ToF_Reset_1, ToF_Reset_2, ToF_Reset_3, ToF_Reset_4, ToF_Reset_5, ToF_Reset_6, ToF_Reset_7
- wire segments 67 -> 66
- no-connect marks 5 -> 4
Changed lines of the file:
@@
 	1    0    0    -1
 $EndComp
-Text HLabel 6000 3100 2    50   Output ~ 0
-ToF_Reset_0
-Text HLabel 6000 3200 2    50   Output ~ 0
-ToF_Reset_1
-Text HLabel 6000 3300 2    50   Output ~ 0
-ToF_Reset_2
-Text HLabel 6000 3400 2    50   Output ~ 0
-ToF_Reset_3
-Text HLabel 6000 3500 2    50   Output ~ 0
-ToF_Reset_4
-Text HLabel 6000 3600 2    50   Output ~ 0
-ToF_Reset_5
-Text HLabel 6000 3700 2    50   Output ~ 0
-ToF_Reset_6
-Text HLabel 6000 3800 2    50   Output ~ 0
-ToF_Reset_7
 Text HLabel 6000 4000 2    50   Output ~ 0
 UART_TX
@@
 Text HLabel 6000 4600 2    50   BiDi ~ 0
 I2C_SCL
-NoConn ~ 4750 4000
-NoConn ~ 4750 4100
-Text HLabel 6000 3900 2    50   Output ~ 0
-TOF_EN
-NoConn ~ 4750 4200
-NoConn ~ 4750 4300
-NoConn ~ 4750 4400
 Text HLabel 4600 4600 0    50   BiDi ~ 0
 I2C_SDA
@@
 L Device:R R9
 U 1 1 5BBDC2CE
-P 4450 4500
-F 0 "R9" V 4243 4500 50  0000 C CNN
-F 1 "R" V 4334 4500 50  0000 C CNN
-F 2 "" V 4380 4500 50  0001 C CNN
-F 3 "~" H 4450 4500 50  0001 C CNN
-	1    4450 4500
-	0    1    1    0
+P 6300 3900
+F 0 "R9" V 6093 3900 50  0000 C CNN
+F 1 "R" V 6184 3900 50  0000 C CNN
+F 2 "" V 6230 3900 50  0001 C CNN
+F 3 "~" H 6300 3900 50  0001 C CNN
+	1    6300 3900
+	0    -1   -1   0
 $EndComp
 $Comp
 L power:GND #PWR026
 U 1 1 5BBDC410
-P 3700 4500
-F 0 "#PWR026" H 3700 4250 50  0001 C CNN
-F 1 "GND" V 3705 4372 50  0000 R CNN
-F 2 "" H 3700 4500 50  0001 C CNN
-F 3 "" H 3700 4500 50  0001 C CNN
-	1    3700 4500
-	0    1    1    0
+P 7050 3900
+F 0 "#PWR026" H 7050 3650 50  0001 C CNN
+F 1 "GND" V 7055 3772 50  0000 R CNN
+F 2 "" H 7050 3900 50  0001 C CNN
+F 3 "" H 7050 3900 50  0001 C CNN
+	1    7050 3900
+	0    -1   -1   0
 $EndComp
 $Comp
 L Device:LED_ALT D6
 U 1 1 5BBDC4BF
-P 4000 4500
-F 0 "D6" H 3991 4716 50  0000 C CNN
-F 1 "LED_ALT" H 3991 4625 50  0000 C CNN
-F 2 "" H 4000 4500 50  0001 C CNN
-F 3 "~" H 4000 4500 50  0001 C CNN
-	1    4000 4500
-	1    0    0    -1
-$EndComp
-Wire Wire Line
-	4600 4500 4750 4500
-Wire Wire Line
-	4150 4500 4300 4500
-Wire Wire Line
-	3700 4500 3850 4500
+P 6750 3900
+F 0 "D6" H 6741 4116 50  0000 C CNN
+F 1 "LED_ALT" H 6741 4025 50  0000 C CNN
+F 2 "" H 6750 3900 50  0001 C CNN
+F 3 "~" H 6750 3900 50  0001 C CNN
+	1    6750 3900
+	-1   0    0    1
+$EndComp
+Wire Wire Line
+	6600 3900 6450 3900
+Wire Wire Line
+	7050 3900 6900 3900
 Wire Wire Line
 	5850 3100 6000 3100
@@
 Wire Wire Line
 	5850 3800 6000 3800
-Wire Wire Line
-	5850 3900 6000 3900
 Wire Wire Line
 	5850 4000 6000 4000
@@
 Wire Wire Line
 	5800 2550 5800 2450
+Wire Wire Line
+	5850 3900 6150 3900
+Text HLabel 6000 3100 2    50   Output ~ 0
+US_TRIG_0
+Text HLabel 6000 3300 2    50   Output ~ 0
+US_TRIG_1
+Text HLabel 6000 3500 2    50   Output ~ 0
+US_TRIG_2
+Text HLabel 6000 3700 2    50   Output ~ 0
+US_TRIG_3
+Text HLabel 6000 3200 2    50   Input ~ 0
+US_ECHO_0
+Text HLabel 6000 3400 2    50   Input ~ 0
+US_ECHO_1
+Text HLabel 6000 3600 2    50   Input ~ 0
+US_ECHO_2
+Text HLabel 6000 3800 2    50   Input ~ 0
+US_ECHO_3
+Text HLabel 4750 4000 0    50   Output ~ 0
+TOF_RESET_DATA
+Text HLabel 4750 4100 0    50   Output ~ 0
+TOF_RESET_SHIFT
+NoConn ~ 4750 4200
+NoConn ~ 4750 4300
+NoConn ~ 4750 4400
+NoConn ~ 4750 4500
 $EndSCHEMATC

Commit message: Added ultrasonic sensors
Parts:
- renumbered R8 to R10, R9 to R11, U5 to U6
Changed lines of the file:
@@
 $Descr A4 11693 8268
 encoding utf-8
-Sheet 3 12
+Sheet 3 16
 Title ""
 Date ""
@@
 $EndDescr
 $Comp
-L MCU_ST_STM32F3:STM32F303K8Tx U5
+L MCU_ST_STM32F3:STM32F303K8Tx U6
 U 1 1 5BBD3F5D
 P 5350 3800
-F 0 "U5" H 5800 2800 50  0000 C CNN
+F 0 "U6" H 5800 2800 50  0000 C CNN
 F 1 "STM32F303K8Tx" H 5800 2700 50  0000 C CNN
 F 2 "Package_QFP:LQFP-32_7x7mm_P0.8mm" H 4850 2900 50  0001 R CNN
@@
 $EndComp
 $Comp
-L power:GND #PWR024
+L power:GND #PWR028
 U 1 1 5BBD4293
 P 3500 3500
-F 0 "#PWR024" H 3500 3250 50  0001 C CNN
+F 0 "#PWR028" H 3500 3250 50  0001 C CNN
 F 1 "GND" V 3505 3372 50  0000 R CNN
 F 2 "" H 3500 3500 50  0001 C CNN
@@
 $EndComp
 $Comp
-L power:GND #PWR025
+L power:GND #PWR029
 U 1 1 5BBD42C5
 P 3500 4000
-F 0 "#PWR025" H 3500 3750 50  0001 C CNN
+F 0 "#PWR029" H 3500 3750 50  0001 C CNN
 F 1 "GND" V 3505 3872 50  0000 R CNN
 F 2 "" H 3500 4000 50  0001 C CNN
@@
 	4100 3950 4100 3900
 $Comp
-L Device:R R8
+L Device:R R10
 U 1 1 5BBD441A
 P 4400 3300
-F 0 "R8" V 4193 3300 50  0000 C CNN
+F 0 "R10" V 4193 3300 50  0000 C CNN
 F 1 "R" V 4284 3300 50  0000 C CNN
 F 2 "" V 4330 3300 50  0001 C CNN
@@
 	4550 3300 4750 3300
 $Comp
-L power:GND #PWR023
+L power:GND #PWR027
 U 1 1 5BBD4A9A
 P 3150 3000
-F 0 "#PWR023" H 3150 2750 50  0001 C CNN
+F 0 "#PWR027" H 3150 2750 50  0001 C CNN
 F 1 "GND" V 3155 2872 50  0000 R CNN
 F 2 "" H 3150 3000 50  0001 C CNN
@@
 	3150 3000 3300 3000
 $Comp
-L power:+3V3 #PWR027
+L power:+3V3 #PWR030
 U 1 1 5BBD4C69
 P 3900 3000
-F 0 "#PWR027" H 3900 2850 50  0001 C CNN
+F 0 "#PWR030" H 3900 2850 50  0001 C CNN
 F 1 "+3V3" V 3915 3128 50  0000 L CNN
 F 2 "" H 3900 3000 50  0001 C CNN
@@
 $EndComp
 $Comp
-L power:GND #PWR028
+L power:GND #PWR031
 U 1 1 5BBD55CA
 P 4650 2500
-F 0 "#PWR028" H 4650 2250 50  0001 C CNN
+F 0 "#PWR031" H 4650 2250 50  0001 C CNN
 F 1 "GND" H 4655 2327 50  0000 C CNN
 F 2 "" H 4650 2500 50  0001 C CNN
@@
 	5350 2650 5450 2650
 $Comp
-L power:+3V3 #PWR033
+L power:+3V3 #PWR036
 U 1 1 5BBD6204
 P 5600 2650
-F 0 "#PWR033" H 5600 2500 50  0001 C CNN
+F 0 "#PWR036" H 5600 2500 50  0001 C CNN
 F 1 "+3V3" V 5615 2778 50  0000 L CNN
 F 2 "" H 5600 2650 50  0001 C CNN
@@
 $EndComp
 $Comp
-L power:GND #PWR034
+L power:GND #PWR037
 U 1 1 5BBD68AE
 P 5800 2050
-F 0 "#PWR034" H 5800 1800 50  0001 C CNN
+F 0 "#PWR037" H 5800 1800 50  0001 C CNN
 F 1 "GND" V 5805 1922 50  0000 R CNN
 F 2 "" H 5800 2050 50  0001 C CNN
@@
 $EndComp
 $Comp
-L power:GND #PWR032
+L power:GND #PWR035
 U 1 1 5BBD68FC
 P 5550 2050
-F 0 "#PWR032" H 5550 1800 50  0001 C CNN
+F 0 "#PWR035" H 5550 1800 50  0001 C CNN
 F 1 "GND" V 5555 1922 50  0000 R CNN
 F 2 "" H 5550 2050 50  0001 C CNN
@@
 $EndComp
 $Comp
-L power:GND #PWR030
+L power:GND #PWR033
 U 1 1 5BBD694A
 P 5300 2050
-F 0 "#PWR030" H 5300 1800 50  0001 C CNN
+F 0 "#PWR033" H 5300 1800 50  0001 C CNN
 F 1 "GND" V 5305 1922 50  0000 R CNN
 F 2 "" H 5300 2050 50  0001 C CNN
@@
 $EndComp
 $Comp
-L power:GND #PWR029
+L power:GND #PWR032
 U 1 1 5BBD6998
 P 5050 2050
-F 0 "#PWR029" H 5050 1800 50  0001 C CNN
+F 0 "#PWR032" H 5050 1800 50  0001 C CNN
 F 1 "GND" V 5055 1922 50  0000 R CNN
 F 2 "" H 5050 2050 50  0001 C CNN
@@
 	5550 2550 5550 2650
 $Comp
-L power:GND #PWR031
+L power:GND #PWR034
 U 1 1 5BBDA4B0
 P 5300 4900
-F 0 "#PWR031" H 5300 4650 50  0001 C CNN
+F 0 "#PWR034" H 5300 4650 50  0001 C CNN
 F 1 "GND" H 5305 4727 50  0000 C CNN
 F 2 "" H 5300 4900 50  0001 C CNN
@@
 Connection ~ 5300 4900
 $Comp
-L Device:R R9
+L Device:R R11
 U 1 1 5BBDC2CE
 P 6300 3900
-F 0 "R9" V 6093 3900 50  0000 C CNN
+F 0 "R11" V 6093 3900 50  0000 C CNN
 F 1 "R" V 6184 3900 50  0000 C CNN
 F 2 "" V 6230 3900 50  0001 C CNN
@@
 $EndComp
 $Comp
-L power:GND #PWR026
+L power:GND #PWR038
 U 1 1 5BBDC410
 P 7050 3900
-F 0 "#PWR026" H 7050 3650 50  0001 C CNN
+F 0 "#PWR038" H 7050 3650 50  0001 C CNN
 F 1 "GND" V 7055 3772 50  0000 R CNN
 F 2 "" H 7050 3900 50  0001 C CNN

Commit message: Fixed shift register voltage translation
Parts:
- renumbered JP1 to JP2, R10 to R8, R11 to R9
Changed lines of the file:
@@
 $Descr A4 11693 8268
 encoding utf-8
-Sheet 3 16
+Sheet 3 19
 Title ""
 Date ""
@@
 $EndComp
 $Comp
-L power:GND #PWR028
+L power:GND #PWR029
 U 1 1 5BBD4293
 P 3500 3500
-F 0 "#PWR028" H 3500 3250 50  0001 C CNN
+F 0 "#PWR029" H 3500 3250 50  0001 C CNN
 F 1 "GND" V 3505 3372 50  0000 R CNN
 F 2 "" H 3500 3500 50  0001 C CNN
@@
 $EndComp
 $Comp
-L power:GND #PWR029
+L power:GND #PWR030
 U 1 1 5BBD42C5
 P 3500 4000
-F 0 "#PWR029" H 3500 3750 50  0001 C CNN
+F 0 "#PWR030" H 3500 3750 50  0001 C CNN
 F 1 "GND" V 3505 3872 50  0000 R CNN
 F 2 "" H 3500 4000 50  0001 C CNN
@@
 	4100 3950 4100 3900
 $Comp
-L Device:R R10
+L Device:R R8
 U 1 1 5BBD441A
 P 4400 3300
-F 0 "R10" V 4193 3300 50  0000 C CNN
+F 0 "R8" V 4193 3300 50  0000 C CNN
 F 1 "R" V 4284 3300 50  0000 C CNN
 F 2 "" V 4330 3300 50  0001 C CNN
@@
 $EndComp
 $Comp
-L Device:Jumper_NC_Dual JP1
+L Device:Jumper_NC_Dual JP2
 U 1 1 5BBD452E
 P 3550 3000
-F 0 "JP1" H 3550 3239 50  0000 C CNN
+F 0 "JP2" H 3550 3239 50  0000 C CNN
 F 1 "Jumper_NC_Dual" H 3550 3148 50  0000 C CNN
 F 2 "" H 3550 3000 50  0001 C CNN
@@
 	4550 3300 4750 3300
 $Comp
-L power:GND #PWR027
+L power:GND #PWR028
 U 1 1 5BBD4A9A
 P 3150 3000
-F 0 "#PWR027" H 3150 2750 50  0001 C CNN
+F 0 "#PWR028" H 3150 2750 50  0001 C CNN
 F 1 "GND" V 3155 2872 50  0000 R CNN
 F 2 "" H 3150 3000 50  0001 C CNN
@@
 	3150 3000 3300 3000
 $Comp
-L power:+3V3 #PWR030
+L power:+3V3 #PWR031
 U 1 1 5BBD4C69
 P 3900 3000
-F 0 "#PWR030" H 3900 2850 50  0001 C CNN
+F 0 "#PWR031" H 3900 2850 50  0001 C CNN
 F 1 "+3V3" V 3915 3128 50  0000 L CNN
 F 2 "" H 3900 3000 50  0001 C CNN
@@
 $EndComp
 $Comp
-L power:GND #PWR031
+L power:GND #PWR032
 U 1 1 5BBD55CA
 P 4650 2500
-F 0 "#PWR031" H 4650 2250 50  0001 C CNN
+F 0 "#PWR032" H 4650 2250 50  0001 C CNN
 F 1 "GND" H 4655 2327 50  0000 C CNN
 F 2 "" H 4650 2500 50  0001 C CNN
@@
 	5350 2650 5450 2650
 $Comp
-L power:+3V3 #PWR036
+L power:+3V3 #PWR037
 U 1 1 5BBD6204
 P 5600 2650
-F 0 "#PWR036" H 5600 2500 50  0001 C CNN
+F 0 "#PWR037" H 5600 2500 50  0001 C CNN
 F 1 "+3V3" V 5615 2778 50  0000 L CNN
 F 2 "" H 5600 2650 50  0001 C CNN
@@
 $EndComp
 $Comp
-L power:GND #PWR037
+L power:GND #PWR038
 U 1 1 5BBD68AE
 P 5800 2050
-F 0 "#PWR037" H 5800 1800 50  0001 C CNN
+F 0 "#PWR038" H 5800 1800 50  0001 C CNN
 F 1 "GND" V 5805 1922 50  0000 R CNN
 F 2 "" H 5800 2050 50  0001 C CNN
@@
 $EndComp
 $Comp
-L power:GND #PWR035
+L power:GND #PWR036
 U 1 1 5BBD68FC
 P 5550 2050
-F 0 "#PWR035" H 5550 1800 50  0001 C CNN
+F 0 "#PWR036" H 5550 1800 50  0001 C CNN
 F 1 "GND" V 5555 1922 50  0000 R CNN
 F 2 "" H 5550 2050 50  0001 C CNN
@@
 $EndComp
 $Comp
-L power:GND #PWR033
+L power:GND #PWR034
 U 1 1 5BBD694A
 P 5300 2050
-F 0 "#PWR033" H 5300 1800 50  0001 C CNN
+F 0 "#PWR034" H 5300 1800 50  0001 C CNN
 F 1 "GND" V 5305 1922 50  0000 R CNN
 F 2 "" H 5300 2050 50  0001 C CNN
@@
 $EndComp
 $Comp
-L power:GND #PWR032
+L power:GND #PWR033
 U 1 1 5BBD6998
 P 5050 2050
-F 0 "#PWR032" H 5050 1800 50  0001 C CNN
+F 0 "#PWR033" H 5050 1800 50  0001 C CNN
 F 1 "GND" V 5055 1922 50  0000 R CNN
 F 2 "" H 5050 2050 50  0001 C CNN
@@
 	5550 2550 5550 2650
 $Comp
-L power:GND #PWR034
+L power:GND #PWR035
 U 1 1 5BBDA4B0
 P 5300 4900
-F 0 "#PWR034" H 5300 4650 50  0001 C CNN
+F 0 "#PWR035" H 5300 4650 50  0001 C CNN
 F 1 "GND" H 5305 4727 50  0000 C CNN
 F 2 "" H 5300 4900 50  0001 C CNN
@@
 Connection ~ 5300 4900
 $Comp
-L Device:R R11
+L Device:R R9
 U 1 1 5BBDC2CE
 P 6300 3900
-F 0 "R11" V 6093 3900 50  0000 C CNN
+F 0 "R9" V 6093 3900 50  0000 C CNN
 F 1 "R" V 6184 3900 50  0000 C CNN
 F 2 "" V 6230 3900 50  0001 C CNN
@@
 $EndComp
 $Comp
-L power:GND #PWR038
+L power:GND #PWR039
 U 1 1 5BBDC410
 P 7050 3900
-F 0 "#PWR038" H 7050 3650 50  0001 C CNN
+F 0 "#PWR039" H 7050 3650 50  0001 C CNN
 F 1 "GND" V 7055 3772 50  0000 R CNN
 F 2 "" H 7050 3900 50  0001 C CNN

Commit message: Fixed TTa pins issue
Connections:
- wire segments 66 -> 62
Other:
- note added: "Pas 5V Tolerant"
Changed lines of the file:
@@
 $Descr A4 11693 8268
 encoding utf-8
-Sheet 3 19
+Sheet 19 19
 Title ""
 Date ""
@@
 	5850 3400 6000 3400
 Wire Wire Line
-	5850 3500 6000 3500
-Wire Wire Line
-	5850 3600 6000 3600
-Wire Wire Line
-	5850 3700 6000 3700
-Wire Wire Line
-	5850 3800 6000 3800
-Wire Wire Line
 	5850 4000 6000 4000
 Wire Wire Line
@@
 Text HLabel 6000 3100 2    50   Output ~ 0
 US_TRIG_0
+Text HLabel 6000 3200 2    50   Output ~ 0
+US_TRIG_1
 Text HLabel 6000 3300 2    50   Output ~ 0
-US_TRIG_1
-Text HLabel 6000 3500 2    50   Output ~ 0
 US_TRIG_2
-Text HLabel 6000 3700 2    50   Output ~ 0
+Text HLabel 6000 3400 2    50   Output ~ 0
 US_TRIG_3
-Text HLabel 6000 3200 2    50   Input ~ 0
+Text HLabel 4750 4200 0    50   Input ~ 0
 US_ECHO_0
-Text HLabel 6000 3400 2    50   Input ~ 0
+Text HLabel 4750 4300 0    50   Input ~ 0
 US_ECHO_1
-Text HLabel 6000 3600 2    50   Input ~ 0
+Text HLabel 4750 4400 0    50   Input ~ 0
 US_ECHO_2
-Text HLabel 6000 3800 2    50   Input ~ 0
+Text HLabel 4750 4500 0    50   Input ~ 0
 US_ECHO_3
 Text HLabel 4750 4000 0    50   Output ~ 0
@@
 Text HLabel 4750 4100 0    50   Output ~ 0
 TOF_RESET_SHIFT
-NoConn ~ 4750 4200
-NoConn ~ 4750 4300
-NoConn ~ 4750 4400
-NoConn ~ 4750 4500
+NoConn ~ 5850 3800
+NoConn ~ 5850 3700
+NoConn ~ 5850 3600
+NoConn ~ 5850 3500
+Text Notes 6550 3250 0    50   ~ 0
+Pas 5V Tolerant
+Wire Notes Line
+	6400 3050 6500 3050
+Wire Notes Line
+	6500 3050 6500 3450
+Wire Notes Line
+	6500 3450 6400 3450
 $EndSCHEMATC
