File: f3.sch (KiCad schematic (older format))
At the start: 13 parts, among them U7 STM32F303K8Tx, Y1 8MHz

Commit message: Update PCB
Parts:
- C10, C9: footprint Capacitor_SMD:C_0805_2012Metric_Pad1.15x1.40mm_HandSolder -> Capacitor_SMD:C_0603_1608Metric_Pad1.05x0.95mm_HandSolder
- Y1: value 8MHz -> 16MHz
Changed lines of the file:
@@
 $Descr A4 11693 8268
 encoding utf-8
-Sheet 15 17
+Sheet 17 17
 Title ""
 Date ""
@@
 F 0 "C9" V 3548 3500 50  0000 C CNN
 F 1 "26p" V 3639 3500 50  0000 C CNN
-F 2 "Capacitor_SMD:C_0805_2012Metric_Pad1.15x1.40mm_HandSolder" H 3838 3350 50  0001 C CNN
+F 2 "Capacitor_SMD:C_0603_1608Metric_Pad1.05x0.95mm_HandSolder" H 3838 3350 50  0001 C CNN
 F 3 "~" H 3800 3500 50  0001 C CNN
 	1    3800 3500
@@
 F 0 "C10" V 3548 4000 50  0000 C CNN
 F 1 "26p" V 3639 4000 50  0000 C CNN
-F 2 "Capacitor_SMD:C_0805_2012Metric_Pad1.15x1.40mm_HandSolder" H 3838 3850 50  0001 C CNN
+F 2 "Capacitor_SMD:C_0603_1608Metric_Pad1.05x0.95mm_HandSolder" H 3838 3850 50  0001 C CNN
 F 3 "~" H 3800 4000 50  0001 C CNN
 	1    3800 4000
@@
 P 4100 3750
 F 0 "Y1" V 4054 3881 50  0000 L CNN
-F 1 "8MHz" V 4145 3881 50  0000 L CNN
+F 1 "16MHz" V 4145 3881 50  0000 L CNN
 F 2 "Crystal:Crystal_HC49-4H_Vertical" H 4100 3750 50  0001 C CNN
 F 3 "~" H 4100 3750 50  0001 C CNN
