File: CAN.sch (KiCad schematic (older format))
At the start: 21 parts, among them P1 CAN_conn, P2 CAN_conn, U1 MCP2551-I-SN, U2 LD1117S33TR_SOT223, U3 LP38693MP-ADJ

Commit message: Added I2C level shifter
Changed lines of the file:
@@
 $Descr A4 11693 8268
 encoding utf-8
-Sheet 2 3
+Sheet 2 4
 Title ""
 Date ""
@@
 Wire Wire Line
 	4050 4600 4050 4500
-Text HLabel 6250 3750 1    50   Input ~ 0
+Text HLabel 6250 3750 1    50   Output ~ 0
 +3V3
 Wire Wire Line

Commit message: Added ToF connectors and fixed schematic ERC
Parts:
- added C3: C, Capacitor_SMD:C_0805_2012Metric_Pad1.15x1.40mm_HandSolder, symbol Device:C
- added D3: LED_ALT, LED_SMD:LED_0805_2012Metric_Castellated, symbol Device:LED_ALT
- added R3: R, Resistor_SMD:R_0805_2012Metric_Pad1.15x1.40mm_HandSolder, symbol Device:R
- added U2: LD1117S50TR_SOT223, Package_TO_SOT_SMD:SOT-223-3_TabPin2, symbol Regulator_Linear:LD1117S50TR_SOT223
- renumbered C3 to C4, C4 to C5, C5 to C6, D3 to D4, D4 to D5, R3 to R4, R4 to R5, R5 to R6, R6 to R7, U2 to U3, U3 to U4
Connections:
- wire segments 67 -> 84
Other:
- moved on the sheet: U3

Commit message: Added ultrasonic sensors
Parts:
- renumbered R1 to R3, R2 to R4, R3 to R5, R4 to R6, R5 to R7, R6 to R8, R7 to R9, U1 to U2, U2 to U3, U3 to U4, U4 to U5
Changed lines of the file:
@@
 $Descr A4 11693 8268
 encoding utf-8
-Sheet 2 12
+Sheet 2 16
 Title ""
 Date ""
@@
 $EndComp
 $Comp
-L power:GND #PWR016
+L power:GND #PWR020
 U 1 1 5B2312B5
 P 6800 2450
-F 0 "#PWR016" H 6800 2200 50  0001 C CNN
+F 0 "#PWR020" H 6800 2200 50  0001 C CNN
 F 1 "GND" H 6805 2277 50  0000 C CNN
 F 2 "" H 6800 2450 50  0001 C CNN
@@
 $EndComp
 $Comp
-L power:GND #PWR012
+L power:GND #PWR016
 U 1 1 5B231C66
 P 5250 2600
-F 0 "#PWR012" H 5250 2350 50  0001 C CNN
+F 0 "#PWR016" H 5250 2350 50  0001 C CNN
 F 1 "GND" H 5255 2427 50  0000 C CNN
 F 2 "" H 5250 2600 50  0001 C CNN
@@
 	5250 2600 5250 2450
 $Comp
-L Interface_CAN_LIN:MCP2551-I-SN U1
+L Interface_CAN_LIN:MCP2551-I-SN U2
 U 1 1 5B231F60
 P 5250 2050
-F 0 "U1" H 5250 2628 50  0000 C CNN
+F 0 "U2" H 5250 2628 50  0000 C CNN
 F 1 "MCP2551-I-SN" H 5250 2537 50  0000 C CNN
 F 2 "Package_SO:SOIC-8_3.9x4.9mm_P1.27mm" H 5250 1550 50  0001 C CIN
@@
 $EndComp
 $Comp
-L power:+5V #PWR011
+L power:+5V #PWR015
 U 1 1 5B232128
 P 5250 1400
-F 0 "#PWR011" H 5250 1250 50  0001 C CNN
+F 0 "#PWR015" H 5250 1250 50  0001 C CNN
 F 1 "+5V" H 5265 1573 50  0000 C CNN
 F 2 "" H 5250 1400 50  0001 C CNN
@@
 	4400 1950 4750 1950
 $Comp
-L Device:R R1
+L Device:R R3
 U 1 1 5B23414E
 P 4350 2550
-F 0 "R1" H 4420 2596 50  0000 L CNN
+F 0 "R3" H 4420 2596 50  0000 L CNN
 F 1 "47kR" H 4420 2505 50  0000 L CNN
 F 2 "Resistor_SMD:R_0805_2012Metric_Pad1.15x1.40mm_HandSolder" V 4280 2550 50  0001 C CNN
@@
 $EndComp
 $Comp
-L power:GND #PWR07
+L power:GND #PWR011
 U 1 1 5B234226
 P 4350 2800
-F 0 "#PWR07" H 4350 2550 50  0001 C CNN
+F 0 "#PWR011" H 4350 2550 50  0001 C CNN
 F 1 "GND" H 4355 2627 50  0000 C CNN
 F 2 "" H 4350 2800 50  0001 C CNN
@@
 AR Path="/5B1D7C42/5BAEB670" Ref="#PWR?"  Part="1"
 AR Path="/5B230D4C/5BAEB670" Ref="#PWR?"  Part="1"
-AR Path="/5BBA64E1/5BAEB670" Ref="#PWR019"  Part="1"
-F 0 "#PWR019" H 8100 4850 50  0001 C CNN
+AR Path="/5BBA64E1/5BAEB670" Ref="#PWR023"  Part="1"
+F 0 "#PWR023" H 8100 4850 50  0001 C CNN
 F 1 "GND" H 8105 4927 50  0000 C CNN
 F 2 "" H 8100 5100 50  0001 C CNN
@@
 AR Path="/5B1D7C42/5BAEB677" Ref="U?"  Part="1"
 AR Path="/5B230D4C/5BAEB677" Ref="U?"  Part="1"
-AR Path="/5BBA64E1/5BAEB677" Ref="U3"  Part="1"
-F 0 "U3" H 7150 4292 50  0000 C CNN
+AR Path="/5BBA64E1/5BAEB677" Ref="U4"  Part="1"
+F 0 "U4" H 7150 4292 50  0000 C CNN
 F 1 "LD1117S33TR_SOT223" H 7150 4201 50  0000 C CNN
 F 2 "Package_TO_SOT_SMD:SOT-223-3_TabPin2" H 7150 4250 50  0001 C CNN
@@
 AR Path="/5B1D7C42/5BAEB68C" Ref="R?"  Part="1"
 AR Path="/5B230D4C/5BAEB68C" Ref="R?"  Part="1"
-AR Path="/5BBA64E1/5BAEB68C" Ref="R4"  Part="1"
-F 0 "R4" H 8170 4896 50  0000 L CNN
+AR Path="/5BBA64E1/5BAEB68C" Ref="R6"  Part="1"
+F 0 "R6" H 8170 4896 50  0000 L CNN
 F 1 "R" H 8170 4805 50  0000 L CNN
 F 2 "Resistor_SMD:R_0805_2012Metric_Pad1.15x1.40mm_HandSolder" V 8030 4850 50  0001 C CNN
@@
 AR Path="/5B1D7C42/5BAEB693" Ref="R?"  Part="1"
 AR Path="/5B230D4C/5BAEB693" Ref="R?"  Part="1"
-AR Path="/5BBA64E1/5BAEB693" Ref="R7"  Part="1"
-F 0 "R7" H 10570 4896 50  0000 L CNN
+AR Path="/5BBA64E1/5BAEB693" Ref="R9"  Part="1"
+F 0 "R9" H 10570 4896 50  0000 L CNN
 F 1 "R" H 10570 4805 50  0000 L CNN
 F 2 "Resistor_SMD:R_0805_2012Metric_Pad1.15x1.40mm_HandSolder" V 10430 4850 50  0001 C CNN
@@
 AR Path="/5B1D7C42/5BAEB69A" Ref="#PWR?"  Part="1"
 AR Path="/5B230D4C/5BAEB69A" Ref="#PWR?"  Part="1"
-AR Path="/5BBA64E1/5BAEB69A" Ref="#PWR022"  Part="1"
-F 0 "#PWR022" H 10500 4900 50  0001 C CNN
+AR Path="/5BBA64E1/5BAEB69A" Ref="#PWR026"  Part="1"
+F 0 "#PWR026" H 10500 4900 50  0001 C CNN
 F 1 "GND" H 10505 4977 50  0000 C CNN
 F 2 "" H 10500 5150 50  0001 C CNN
@@
 AR Path="/5B1D7C42/5BAEB6A0" Ref="#PWR?"  Part="1"
 AR Path="/5B230D4C/5BAEB6A0" Ref="#PWR?"  Part="1"
-AR Path="/5BBA64E1/5BAEB6A0" Ref="#PWR020"  Part="1"
-F 0 "#PWR020" H 9100 4400 50  0001 C CNN
+AR Path="/5BBA64E1/5BAEB6A0" Ref="#PWR024"  Part="1"
+F 0 "#PWR024" H 9100 4400 50  0001 C CNN
 F 1 "GND" H 9105 4477 50  0000 C CNN
 F 2 "" H 9100 4650 50  0001 C CNN
@@
 AR Path="/5B1D7C42/5BAEB6B4" Ref="#PWR?"  Part="1"
 AR Path="/5B230D4C/5BAEB6B4" Ref="#PWR?"  Part="1"
-AR Path="/5BBA64E1/5BAEB6B4" Ref="#PWR09"  Part="1"
-F 0 "#PWR09" H 4500 4500 50  0001 C CNN
+AR Path="/5BBA64E1/5BAEB6B4" Ref="#PWR013"  Part="1"
+F 0 "#PWR013" H 4500 4500 50  0001 C CNN
 F 1 "GND" H 4505 4577 50  0000 C CNN
 F 2 "" H 4500 4750 50  0001 C CNN
@@
 AR Path="/5B1D7C42/5BAEB6E4" Ref="#PWR?"  Part="1"
 AR Path="/5B230D4C/5BAEB6E4" Ref="#PWR?"  Part="1"
-AR Path="/5BBA64E1/5BAEB6E4" Ref="#PWR06"  Part="1"
-F 0 "#PWR06" H 4050 4350 50  0001 C CNN
+AR Path="/5BBA64E1/5BAEB6E4" Ref="#PWR010"  Part="1"
+F 0 "#PWR010" H 4050 4350 50  0001 C CNN
 F 1 "GND" H 4055 4427 50  0000 C CNN
 F 2 "" H 4050 4600 50  0001 C CNN
@@
 AR Path="/5B1D7C42/5BAEB705" Ref="R?"  Part="1"
 AR Path="/5B230D4C/5BAEB705" Ref="R?"  Part="1"
-AR Path="/5BBA64E1/5BAEB705" Ref="R2"  Part="1"
-F 0 "R2" H 5070 4896 50  0000 L CNN
+AR Path="/5BBA64E1/5BAEB705" Ref="R4"  Part="1"
+F 0 "R4" H 5070 4896 50  0000 L CNN
 F 1 "R" H 5070 4805 50  0000 L CNN
 F 2 "Resistor_SMD:R_0805_2012Metric_Pad1.15x1.40mm_HandSolder" V 4930 4850 50  0001 C CNN
@@
 AR Path="/5B1D7C42/5BAEB70C" Ref="#PWR?"  Part="1"
 AR Path="/5B230D4C/5BAEB70C" Ref="#PWR?"  Part="1"
-AR Path="/5BBA64E1/5BAEB70C" Ref="#PWR010"  Part="1"
-F 0 "#PWR010" H 5000 4900 50  0001 C CNN
+AR Path="/5BBA64E1/5BAEB70C" Ref="#PWR014"  Part="1"
+F 0 "#PWR014" H 5000 4900 50  0001 C CNN
 F 1 "GND" H 5005 4977 50  0000 C CNN
 F 2 "" H 5000 5150 50  0001 C CNN
@@
 AR Path="/5B1D7C42/5BAEB712" Ref="#PWR?"  Part="1"
 AR Path="/5B230D4C/5BAEB712" Ref="#PWR?"  Part="1"
-AR Path="/5BBA64E1/5BAEB712" Ref="#PWR018"  Part="1"
-F 0 "#PWR018" H 7650 4800 50  0001 C CNN
+AR Path="/5BBA64E1/5BAEB712" Ref="#PWR022"  Part="1"
+F 0 "#PWR022" H 7650 4800 50  0001 C CNN
 F 1 "GND" H 7655 4877 50  0000 C CNN
 F 2 "" H 7650 5050 50  0001 C CNN
@@
 AR Path="/5B1D7C42/5BAEB724" Ref="#PWR?"  Part="1"
 AR Path="/5B230D4C/5BAEB724" Ref="#PWR?"  Part="1"
-AR Path="/5BBA64E1/5BAEB724" Ref="#PWR017"  Part="1"
-F 0 "#PWR017" H 7150 4250 50  0001 C CNN
+AR Path="/5BBA64E1/5BAEB724" Ref="#PWR021"  Part="1"
+F 0 "#PWR021" H 7150 4250 50  0001 C CNN
 F 1 "GND" H 7155 4327 50  0000 C CNN
 F 2 "" H 7150 4500 50  0001 C CNN
@@
 $EndComp
 $Comp
-L power:GND #PWR08
+L power:GND #PWR012
 U 1 1 5BB50F49
 P 4400 1550
-F 0 "#PWR08" H 4400 1300 50  0001 C CNN
+F 0 "#PWR012" H 4400 1300 50  0001 C CNN
 F 1 "GND" V 4405 1422 50  0000 R CNN
 F 2 "" H 4400 1550 50  0001 C CNN
@@
 Connection ~ 7650 4050
 $Comp
-L PhoenixRobotik:LP38693MP-ADJ U4
+L PhoenixRobotik:LP38693MP-ADJ U5
 U 1 1 5BBAAF8D
 P 9100 4150
-F 0 "U4" H 9100 4517 50  0000 C CNN
+F 0 "U5" H 9100 4517 50  0000 C CNN
 F 1 "LP38693MP-ADJ" H 9100 4426 50  0000 C CNN
 F 2 "" H 9100 4150 50  0001 C CNN
@@
 Connection ~ 9100 4550
 $Comp
-L Device:R R5
+L Device:R R7
 U 1 1 5BBBEE12
 P 9600 4350
-F 0 "R5" H 9670 4396 50  0000 L CNN
+F 0 "R7" H 9670 4396 50  0000 L CNN
 F 1 "R2" H 9670 4305 50  0000 L CNN
 F 2 "" V 9530 4350 50  0001 C CNN
@@
 $EndComp
 $Comp
-L Device:R R6
+L Device:R R8
 U 1 1 5BBBEE87
 P 9900 4150
-F 0 "R6" V 9693 4150 50  0000 C CNN
+F 0 "R8" V 9693 4150 50  0000 C CNN
 F 1 "R1" V 9784 4150 50  0000 C CNN
 F 2 "" V 9830 4150 50  0001 C CNN
@@
 	10200 4150 10200 4200
 $Comp
-L power:GND #PWR021
+L power:GND #PWR025
 U 1 1 5BBC2CE7
 P 10200 4650
-F 0 "#PWR021" H 10200 4400 50  0001 C CNN
+F 0 "#PWR025" H 10200 4400 50  0001 C CNN
 F 1 "GND" H 10205 4477 50  0000 C CNN
 F 2 "" H 10200 4650 50  0001 C CNN
@@
 AR Path="/5B1D7C42/5BBE78B6" Ref="#PWR?"  Part="1"
 AR Path="/5B230D4C/5BBE78B6" Ref="#PWR?"  Part="1"
-AR Path="/5BBA64E1/5BBE78B6" Ref="#PWR015"  Part="1"
-F 0 "#PWR015" H 6450 4850 50  0001 C CNN
+AR Path="/5BBA64E1/5BBE78B6" Ref="#PWR019"  Part="1"
+F 0 "#PWR019" H 6450 4850 50  0001 C CNN
 F 1 "GND" H 6455 4927 50  0000 C CNN
 F 2 "" H 6450 5100 50  0001 C CNN
@@
 AR Path="/5B1D7C42/5BBE78C2" Ref="R?"  Part="1"
 AR Path="/5B230D4C/5BBE78C2" Ref="R?"  Part="1"
-AR Path="/5BBA64E1/5BBE78C2" Ref="R3"  Part="1"
-F 0 "R3" H 6520 4896 50  0000 L CNN
+AR Path="/5BBA64E1/5BBE78C2" Ref="R5"  Part="1"
+F 0 "R5" H 6520 4896 50  0000 L CNN
 F 1 "R" H 6520 4805 50  0000 L CNN
 F 2 "Resistor_SMD:R_0805_2012Metric_Pad1.15x1.40mm_HandSolder" V 6380 4850 50  0001 C CNN
@@
 AR Path="/5B1D7C42/5BBE78D1" Ref="#PWR?"  Part="1"
 AR Path="/5B230D4C/5BBE78D1" Ref="#PWR?"  Part="1"
-AR Path="/5BBA64E1/5BBE78D1" Ref="#PWR014"  Part="1"
-F 0 "#PWR014" H 6000 4800 50  0001 C CNN
+AR Path="/5BBA64E1/5BBE78D1" Ref="#PWR018"  Part="1"
+F 0 "#PWR018" H 6000 4800 50  0001 C CNN
 F 1 "GND" H 6005 4877 50  0000 C CNN
 F 2 "" H 6000 5050 50  0001 C CNN
@@
 Connection ~ 6450 4050
 $Comp
-L Regulator_Linear:LD1117S50TR_SOT223 U2
+L Regulator_Linear:LD1117S50TR_SOT223 U3
 U 1 1 5BBEAC6A
 P 5500 4050
-F 0 "U2" H 5500 4292 50  0000 C CNN
+F 0 "U3" H 5500 4292 50  0000 C CNN
 F 1 "LD1117S50TR_SOT223" H 5500 4201 50  0000 C CNN
 F 2 "Package_TO_SOT_SMD:SOT-223-3_TabPin2" H 5500 4250 50  0001 C CNN
@@
 Connection ~ 5000 4050
 $Comp
-L power:GND #PWR013
+L power:GND #PWR017
 U 1 1 5BBEDDC3
 P 5500 4500
-F 0 "#PWR013" H 5500 4250 50  0001 C CNN
+F 0 "#PWR017" H 5500 4250 50  0001 C CNN
 F 1 "GND" H 5505 4327 50  0000 C CNN
 F 2 "" H 5500 4500 50  0001 C CNN

Commit message: Fixed shift register voltage translation
Parts:
- renumbered R3 to R1, R4 to R2, R5 to R3, R6 to R4, R7 to R5, R8 to R6, R9 to R7
Changed lines of the file:
@@
 $Descr A4 11693 8268
 encoding utf-8
-Sheet 2 16
+Sheet 2 19
 Title ""
 Date ""
@@
 $EndComp
 $Comp
-L power:GND #PWR020
+L power:GND #PWR021
 U 1 1 5B2312B5
 P 6800 2450
-F 0 "#PWR020" H 6800 2200 50  0001 C CNN
+F 0 "#PWR021" H 6800 2200 50  0001 C CNN
 F 1 "GND" H 6805 2277 50  0000 C CNN
 F 2 "" H 6800 2450 50  0001 C CNN
@@
 $EndComp
 $Comp
-L power:GND #PWR016
+L power:GND #PWR017
 U 1 1 5B231C66
 P 5250 2600
-F 0 "#PWR016" H 5250 2350 50  0001 C CNN
+F 0 "#PWR017" H 5250 2350 50  0001 C CNN
 F 1 "GND" H 5255 2427 50  0000 C CNN
 F 2 "" H 5250 2600 50  0001 C CNN
@@
 $EndComp
 $Comp
-L power:+5V #PWR015
+L power:+5V #PWR016
 U 1 1 5B232128
 P 5250 1400
-F 0 "#PWR015" H 5250 1250 50  0001 C CNN
+F 0 "#PWR016" H 5250 1250 50  0001 C CNN
 F 1 "+5V" H 5265 1573 50  0000 C CNN
 F 2 "" H 5250 1400 50  0001 C CNN
@@
 	4400 1950 4750 1950
 $Comp
-L Device:R R3
+L Device:R R1
 U 1 1 5B23414E
 P 4350 2550
-F 0 "R3" H 4420 2596 50  0000 L CNN
+F 0 "R1" H 4420 2596 50  0000 L CNN
 F 1 "47kR" H 4420 2505 50  0000 L CNN
 F 2 "Resistor_SMD:R_0805_2012Metric_Pad1.15x1.40mm_HandSolder" V 4280 2550 50  0001 C CNN
@@
 $EndComp
 $Comp
-L power:GND #PWR011
+L power:GND #PWR012
 U 1 1 5B234226
 P 4350 2800
-F 0 "#PWR011" H 4350 2550 50  0001 C CNN
+F 0 "#PWR012" H 4350 2550 50  0001 C CNN
 F 1 "GND" H 4355 2627 50  0000 C CNN
 F 2 "" H 4350 2800 50  0001 C CNN
@@
 AR Path="/5B1D7C42/5BAEB670" Ref="#PWR?"  Part="1"
 AR Path="/5B230D4C/5BAEB670" Ref="#PWR?"  Part="1"
-AR Path="/5BBA64E1/5BAEB670" Ref="#PWR023"  Part="1"
-F 0 "#PWR023" H 8100 4850 50  0001 C CNN
+AR Path="/5BBA64E1/5BAEB670" Ref="#PWR024"  Part="1"
+F 0 "#PWR024" H 8100 4850 50  0001 C CNN
 F 1 "GND" H 8105 4927 50  0000 C CNN
 F 2 "" H 8100 5100 50  0001 C CNN
@@
 AR Path="/5B1D7C42/5BAEB68C" Ref="R?"  Part="1"
 AR Path="/5B230D4C/5BAEB68C" Ref="R?"  Part="1"
-AR Path="/5BBA64E1/5BAEB68C" Ref="R6"  Part="1"
-F 0 "R6" H 8170 4896 50  0000 L CNN
+AR Path="/5BBA64E1/5BAEB68C" Ref="R4"  Part="1"
+F 0 "R4" H 8170 4896 50  0000 L CNN
 F 1 "R" H 8170 4805 50  0000 L CNN
 F 2 "Resistor_SMD:R_0805_2012Metric_Pad1.15x1.40mm_HandSolder" V 8030 4850 50  0001 C CNN
@@
 AR Path="/5B1D7C42/5BAEB693" Ref="R?"  Part="1"
 AR Path="/5B230D4C/5BAEB693" Ref="R?"  Part="1"
-AR Path="/5BBA64E1/5BAEB693" Ref="R9"  Part="1"
-F 0 "R9" H 10570 4896 50  0000 L CNN
+AR Path="/5BBA64E1/5BAEB693" Ref="R7"  Part="1"
+F 0 "R7" H 10570 4896 50  0000 L CNN
 F 1 "R" H 10570 4805 50  0000 L CNN
 F 2 "Resistor_SMD:R_0805_2012Metric_Pad1.15x1.40mm_HandSolder" V 10430 4850 50  0001 C CNN
@@
 AR Path="/5B1D7C42/5BAEB69A" Ref="#PWR?"  Part="1"
 AR Path="/5B230D4C/5BAEB69A" Ref="#PWR?"  Part="1"
-AR Path="/5BBA64E1/5BAEB69A" Ref="#PWR026"  Part="1"
-F 0 "#PWR026" H 10500 4900 50  0001 C CNN
+AR Path="/5BBA64E1/5BAEB69A" Ref="#PWR027"  Part="1"
+F 0 "#PWR027" H 10500 4900 50  0001 C CNN
 F 1 "GND" H 10505 4977 50  0000 C CNN
 F 2 "" H 10500 5150 50  0001 C CNN
@@
 AR Path="/5B1D7C42/5BAEB6A0" Ref="#PWR?"  Part="1"
 AR Path="/5B230D4C/5BAEB6A0" Ref="#PWR?"  Part="1"
-AR Path="/5BBA64E1/5BAEB6A0" Ref="#PWR024"  Part="1"
-F 0 "#PWR024" H 9100 4400 50  0001 C CNN
+AR Path="/5BBA64E1/5BAEB6A0" Ref="#PWR025"  Part="1"
+F 0 "#PWR025" H 9100 4400 50  0001 C CNN
 F 1 "GND" H 9105 4477 50  0000 C CNN
 F 2 "" H 9100 4650 50  0001 C CNN
@@
 AR Path="/5B1D7C42/5BAEB6B4" Ref="#PWR?"  Part="1"
 AR Path="/5B230D4C/5BAEB6B4" Ref="#PWR?"  Part="1"
-AR Path="/5BBA64E1/5BAEB6B4" Ref="#PWR013"  Part="1"
-F 0 "#PWR013" H 4500 4500 50  0001 C CNN
+AR Path="/5BBA64E1/5BAEB6B4" Ref="#PWR014"  Part="1"
+F 0 "#PWR014" H 4500 4500 50  0001 C CNN
 F 1 "GND" H 4505 4577 50  0000 C CNN
 F 2 "" H 4500 4750 50  0001 C CNN
@@
 AR Path="/5B1D7C42/5BAEB6E4" Ref="#PWR?"  Part="1"
 AR Path="/5B230D4C/5BAEB6E4" Ref="#PWR?"  Part="1"
-AR Path="/5BBA64E1/5BAEB6E4" Ref="#PWR010"  Part="1"
-F 0 "#PWR010" H 4050 4350 50  0001 C CNN
+AR Path="/5BBA64E1/5BAEB6E4" Ref="#PWR011"  Part="1"
+F 0 "#PWR011" H 4050 4350 50  0001 C CNN
 F 1 "GND" H 4055 4427 50  0000 C CNN
 F 2 "" H 4050 4600 50  0001 C CNN
@@
 AR Path="/5B1D7C42/5BAEB705" Ref="R?"  Part="1"
 AR Path="/5B230D4C/5BAEB705" Ref="R?"  Part="1"
-AR Path="/5BBA64E1/5BAEB705" Ref="R4"  Part="1"
-F 0 "R4" H 5070 4896 50  0000 L CNN
+AR Path="/5BBA64E1/5BAEB705" Ref="R2"  Part="1"
+F 0 "R2" H 5070 4896 50  0000 L CNN
 F 1 "R" H 5070 4805 50  0000 L CNN
 F 2 "Resistor_SMD:R_0805_2012Metric_Pad1.15x1.40mm_HandSolder" V 4930 4850 50  0001 C CNN
@@
 AR Path="/5B1D7C42/5BAEB70C" Ref="#PWR?"  Part="1"
 AR Path="/5B230D4C/5BAEB70C" Ref="#PWR?"  Part="1"
-AR Path="/5BBA64E1/5BAEB70C" Ref="#PWR014"  Part="1"
-F 0 "#PWR014" H 5000 4900 50  0001 C CNN
+AR Path="/5BBA64E1/5BAEB70C" Ref="#PWR015"  Part="1"
+F 0 "#PWR015" H 5000 4900 50  0001 C CNN
 F 1 "GND" H 5005 4977 50  0000 C CNN
 F 2 "" H 5000 5150 50  0001 C CNN
@@
 AR Path="/5B1D7C42/5BAEB712" Ref="#PWR?"  Part="1"
 AR Path="/5B230D4C/5BAEB712" Ref="#PWR?"  Part="1"
-AR Path="/5BBA64E1/5BAEB712" Ref="#PWR022"  Part="1"
-F 0 "#PWR022" H 7650 4800 50  0001 C CNN
+AR Path="/5BBA64E1/5BAEB712" Ref="#PWR023"  Part="1"
+F 0 "#PWR023" H 7650 4800 50  0001 C CNN
 F 1 "GND" H 7655 4877 50  0000 C CNN
 F 2 "" H 7650 5050 50  0001 C CNN
@@
 AR Path="/5B1D7C42/5BAEB724" Ref="#PWR?"  Part="1"
 AR Path="/5B230D4C/5BAEB724" Ref="#PWR?"  Part="1"
-AR Path="/5BBA64E1/5BAEB724" Ref="#PWR021"  Part="1"
-F 0 "#PWR021" H 7150 4250 50  0001 C CNN
+AR Path="/5BBA64E1/5BAEB724" Ref="#PWR022"  Part="1"
+F 0 "#PWR022" H 7150 4250 50  0001 C CNN
 F 1 "GND" H 7155 4327 50  0000 C CNN
 F 2 "" H 7150 4500 50  0001 C CNN
@@
 $EndComp
 $Comp
-L power:GND #PWR012
+L power:GND #PWR013
 U 1 1 5BB50F49
 P 4400 1550
-F 0 "#PWR012" H 4400 1300 50  0001 C CNN
+F 0 "#PWR013" H 4400 1300 50  0001 C CNN
 F 1 "GND" V 4405 1422 50  0000 R CNN
 F 2 "" H 4400 1550 50  0001 C CNN
@@
 Connection ~ 9100 4550
 $Comp
-L Device:R R7
+L Device:R R5
 U 1 1 5BBBEE12
 P 9600 4350
-F 0 "R7" H 9670 4396 50  0000 L CNN
+F 0 "R5" H 9670 4396 50  0000 L CNN
 F 1 "R2" H 9670 4305 50  0000 L CNN
 F 2 "" V 9530 4350 50  0001 C CNN
@@
 $EndComp
 $Comp
-L Device:R R8
+L Device:R R6
 U 1 1 5BBBEE87
 P 9900 4150
-F 0 "R8" V 9693 4150 50  0000 C CNN
+F 0 "R6" V 9693 4150 50  0000 C CNN
 F 1 "R1" V 9784 4150 50  0000 C CNN
 F 2 "" V 9830 4150 50  0001 C CNN
@@
 	10200 4150 10200 4200
 $Comp
-L power:GND #PWR025
+L power:GND #PWR026
 U 1 1 5BBC2CE7
 P 10200 4650
-F 0 "#PWR025" H 10200 4400 50  0001 C CNN
+F 0 "#PWR026" H 10200 4400 50  0001 C CNN
 F 1 "GND" H 10205 4477 50  0000 C CNN
 F 2 "" H 10200 4650 50  0001 C CNN
@@
 AR Path="/5B1D7C42/5BBE78B6" Ref="#PWR?"  Part="1"
 AR Path="/5B230D4C/5BBE78B6" Ref="#PWR?"  Part="1"
-AR Path="/5BBA64E1/5BBE78B6" Ref="#PWR019"  Part="1"
-F 0 "#PWR019" H 6450 4850 50  0001 C CNN
+AR Path="/5BBA64E1/5BBE78B6" Ref="#PWR020"  Part="1"
+F 0 "#PWR020" H 6450 4850 50  0001 C CNN
 F 1 "GND" H 6455 4927 50  0000 C CNN
 F 2 "" H 6450 5100 50  0001 C CNN
@@
 AR Path="/5B1D7C42/5BBE78C2" Ref="R?"  Part="1"
 AR Path="/5B230D4C/5BBE78C2" Ref="R?"  Part="1"
-AR Path="/5BBA64E1/5BBE78C2" Ref="R5"  Part="1"
-F 0 "R5" H 6520 4896 50  0000 L CNN
+AR Path="/5BBA64E1/5BBE78C2" Ref="R3"  Part="1"
+F 0 "R3" H 6520 4896 50  0000 L CNN
 F 1 "R" H 6520 4805 50  0000 L CNN
 F 2 "Resistor_SMD:R_0805_2012Metric_Pad1.15x1.40mm_HandSolder" V 6380 4850 50  0001 C CNN
@@
 AR Path="/5B1D7C42/5BBE78D1" Ref="#PWR?"  Part="1"
 AR Path="/5B230D4C/5BBE78D1" Ref="#PWR?"  Part="1"
-AR Path="/5BBA64E1/5BBE78D1" Ref="#PWR018"  Part="1"
-F 0 "#PWR018" H 6000 4800 50  0001 C CNN
+AR Path="/5BBA64E1/5BBE78D1" Ref="#PWR019"  Part="1"
+F 0 "#PWR019" H 6000 4800 50  0001 C CNN
 F 1 "GND" H 6005 4877 50  0000 C CNN
 F 2 "" H 6000 5050 50  0001 C CNN
@@
 Connection ~ 5000 4050
 $Comp
-L power:GND #PWR017
+L power:GND #PWR018
 U 1 1 5BBEDDC3
 P 5500 4500
-F 0 "#PWR017" H 5500 4250 50  0001 C CNN
+F 0 "#PWR018" H 5500 4250 50  0001 C CNN
 F 1 "GND" H 5505 4327 50  0000 C CNN
 F 2 "" H 5500 4500 50  0001 C CNN

Commit message: Added IC for level translation with ultrasonic sensors
Parts:
- C7: renamed from C5; footprint (none) -> Capacitor_SMD:C_0805_2012Metric_Pad1.15x1.40mm_HandSolder
- C8: renamed from C6; footprint (none) -> Capacitor_SMD:C_0805_2012Metric_Pad1.15x1.40mm_HandSolder
- R6: renamed from R5; footprint (none) -> Resistor_SMD:R_0805_2012Metric_Pad1.15x1.40mm_HandSolder
- R7: renamed from R6; footprint (none) -> Resistor_SMD:R_0805_2012Metric_Pad1.15x1.40mm_HandSolder
- renumbered C1 to C3, C2 to C4, C3 to C5, C4 to C6, R1 to R2, R2 to R3, R3 to R4, R4 to R5, R7 to R8, U2 to U3, U3 to U4, U4 to U5, U5 to U6

Commit message: Footprint association
Parts:
- C4: footprint Capacitor_SMD:C_0805_2012Metric_Pad1.33x1.40mm_HandSolder -> Capacitor_SMD:C_0805_2012Metric_Pad1.15x1.40mm_HandSolder
- P1, P2: footprint Connector_Molex:Molex_KK-254_AE-6410-04A_1x04_P2.54mm_Vertical -> Connector_JST:JST_XH_B04B-XH-A_1x04_P2.50mm_Vertical
- U6: footprint (none) -> Package_TO_SOT_SMD:SOT-223-5
Changed lines of the file:
@@
 F 0 "P1" H 6500 1750 50  0000 L CNN
 F 1 "CAN_conn" H 6450 2350 50  0000 L CNN
-F 2 "Connector_Molex:Molex_KK-254_AE-6410-04A_1x04_P2.54mm_Vertical" H 6850 1700 50  0001 C CNN
+F 2 "Connector_JST:JST_XH_B04B-XH-A_1x04_P2.50mm_Vertical" H 6850 1700 50  0001 C CNN
 F 3 "https://github.com/PhenixRobotik/phenix_kicad" H 7149 1959 50  0001 L CNN
 	1    6700 2050
@@
 F 0 "P2" H 7250 1750 50  0000 L CNN
 F 1 "CAN_conn" H 7200 2350 50  0000 L CNN
-F 2 "Connector_Molex:Molex_KK-254_AE-6410-04A_1x04_P2.54mm_Vertical" H 7600 1700 50  0001 C CNN
+F 2 "Connector_JST:JST_XH_B04B-XH-A_1x04_P2.50mm_Vertical" H 7600 1700 50  0001 C CNN
 F 3 "https://github.com/PhenixRobotik/phenix_kicad" H 7899 1959 50  0001 L CNN
 	1    7450 2050
@@
 F 0 "C4" V 4398 1550 50  0000 C CNN
 F 1 "100nF" V 4489 1550 50  0000 C CNN
-F 2 "Capacitor_SMD:C_0805_2012Metric_Pad1.33x1.40mm_HandSolder" H 4688 1400 50  0001 C CNN
+F 2 "Capacitor_SMD:C_0805_2012Metric_Pad1.15x1.40mm_HandSolder" H 4688 1400 50  0001 C CNN
 F 3 "~" H 4650 1550 50  0001 C CNN
 	1    4650 1550
@@
 F 0 "U6" H 9100 4517 50  0000 C CNN
 F 1 "LP38693MP-ADJ" H 9100 4426 50  0000 C CNN
-F 2 "" H 9100 4150 50  0001 C CNN
+F 2 "Package_TO_SOT_SMD:SOT-223-5" H 9100 4150 50  0001 C CNN
 F 3 "http://www.ti.com/lit/ds/snvs324k/snvs324k.pdf" H 9100 4150 50  0001 C CNN
 	1    9100 4150
