File: CAN.sch (KiCad schematic (older format))
At the start: 25 parts, among them P1 CAN_conn, P2 CAN_conn, U3 TCAN332, U4 LD1117S50TR_SOT223, U5 LD1117S33TR_SOT223, U6 LP38693MP-ADJ

Commit message: Update PCB
Parts:
- D1: footprint Diode_SMD:D_2114_3652Metric_Castellated -> Diode_SMD:D_SMA
Changed lines of the file:
@@
 $Descr A4 11693 8268
 encoding utf-8
-Sheet 17 17
+Sheet 16 17
 Title ""
 Date ""
@@
 F 0 "D1" V 2804 4429 50  0000 L CNN
 F 1 "D" V 2895 4429 50  0000 L CNN
-F 2 "Diode_SMD:D_2114_3652Metric_Castellated" H 2850 4350 50  0001 C CNN
+F 2 "Diode_SMD:D_SMA" H 2850 4350 50  0001 C CNN
 F 3 "~" H 2850 4350 50  0001 C CNN
 F 4 "743-5961" V 2850 4350 50  0001 C CNN "RS"
