File: I2C.sch (KiCad schematic (older format))
At the start: 6 parts

Commit message: Added ToF connectors and fixed schematic ERC
Parts:
- gave numbers to parts that had none: 6
Changed lines of the file:
@@
 $EndDescr
 $Comp
-L Transistor_FET:BSS138 Q?
+L Transistor_FET:BSS138 Q1
 U 1 1 5BBBF528
 P 2850 3300
-F 0 "Q?" V 3193 3300 50  0000 C CNN
+F 0 "Q1" V 3193 3300 50  0000 C CNN
 F 1 "BSS138" V 3102 3300 50  0000 C CNN
 F 2 "Package_TO_SOT_SMD:SOT-23" H 3050 3225 50  0001 L CIN
@@
 I2C_STM32_SDA
 $Comp
-L Transistor_FET:BSS138 Q?
+L Transistor_FET:BSS138 Q2
 U 1 1 5BBBF64A
 P 3400 3700
-F 0 "Q?" V 3743 3700 50  0000 C CNN
+F 0 "Q2" V 3743 3700 50  0000 C CNN
 F 1 "BSS138" V 3652 3700 50  0000 C CNN
 F 2 "Package_TO_SOT_SMD:SOT-23" H 3600 3625 50  0001 L CIN
@@
 $EndComp
 $Comp
-L power:+3.3V #PWR?
+L power:+3.3V #PWR051
 U 1 1 5BBBF787
 P 2450 2650
-F 0 "#PWR?" H 2450 2500 50  0001 C CNN
+F 0 "#PWR051" H 2450 2500 50  0001 C CNN
 F 1 "+3.3V" H 2465 2823 50  0000 C CNN
 F 2 "" H 2450 2650 50  0001 C CNN
@@
 $EndComp
 $Comp
-L power:+2V8 #PWR?
+L power:+2V8 #PWR052
 U 1 1 5BBBFBE8
 P 2700 3950
-F 0 "#PWR?" H 2700 3800 50  0001 C CNN
+F 0 "#PWR052" H 2700 3800 50  0001 C CNN
 F 1 "+2V8" V 2715 4078 50  0000 L CNN
 F 2 "" H 2700 3950 50  0001 C CNN
@@
 $EndComp
 $Comp
-L Device:R R?
+L Device:R R10
 U 1 1 5BBBFC54
 P 2200 3450
-F 0 "R?" H 2270 3496 50  0000 L CNN
+F 0 "R10" H 2270 3496 50  0000 L CNN
 F 1 "R" H 2270 3405 50  0000 L CNN
 F 2 "" V 2130 3450 50  0001 C CNN
@@
 $EndComp
 $Comp
-L Device:R R?
+L Device:R R11
 U 1 1 5BBBFCA5
 P 2450 3050
-F 0 "R?" H 2520 3096 50  0000 L CNN
+F 0 "R11" H 2520 3096 50  0000 L CNN
 F 1 "R" H 2520 3005 50  0000 L CNN
 F 2 "" V 2380 3050 50  0001 C CNN
@@
 	3400 3950 3400 3900
 $Comp
-L Device:R R?
+L Device:R R12
 U 1 1 5BBC053E
 P 3800 3350
-F 0 "R?" H 3870 3396 50  0000 L CNN
+F 0 "R12" H 3870 3396 50  0000 L CNN
 F 1 "R" H 3870 3305 50  0000 L CNN
 F 2 "" V 3730 3350 50  0001 C CNN
@@
 $EndComp
 $Comp
-L Device:R R?
+L Device:R R13
 U 1 1 5BBC057D
 P 4050 3750
-F 0 "R?" H 4120 3796 50  0000 L CNN
+F 0 "R13" H 4120 3796 50  0000 L CNN
 F 1 "R" H 4120 3705 50  0000 L CNN
 F 2 "" V 3980 3750 50  0001 C CNN

Commit message: Added ultrasonic sensors
Parts:
- renumbered Q1 to Q2, Q2 to Q3, R10 to R12, R11 to R13, R12 to R14, R13 to R15
Changed lines of the file:
@@
 $Descr A4 11693 8268
 encoding utf-8
-Sheet 4 12
+Sheet 4 16
 Title ""
 Date ""
@@
 $EndDescr
 $Comp
-L Transistor_FET:BSS138 Q1
+L Transistor_FET:BSS138 Q2
 U 1 1 5BBBF528
 P 2850 3300
-F 0 "Q1" V 3193 3300 50  0000 C CNN
+F 0 "Q2" V 3193 3300 50  0000 C CNN
 F 1 "BSS138" V 3102 3300 50  0000 C CNN
 F 2 "Package_TO_SOT_SMD:SOT-23" H 3050 3225 50  0001 L CIN
@@
 I2C_STM32_SDA
 $Comp
-L Transistor_FET:BSS138 Q2
+L Transistor_FET:BSS138 Q3
 U 1 1 5BBBF64A
 P 3400 3700
-F 0 "Q2" V 3743 3700 50  0000 C CNN
+F 0 "Q3" V 3743 3700 50  0000 C CNN
 F 1 "BSS138" V 3652 3700 50  0000 C CNN
 F 2 "Package_TO_SOT_SMD:SOT-23" H 3600 3625 50  0001 L CIN
@@
 $EndComp
 $Comp
-L power:+3.3V #PWR035
+L power:+3.3V #PWR039
 U 1 1 5BBBF787
 P 2450 2650
-F 0 "#PWR035" H 2450 2500 50  0001 C CNN
+F 0 "#PWR039" H 2450 2500 50  0001 C CNN
 F 1 "+3.3V" H 2465 2823 50  0000 C CNN
 F 2 "" H 2450 2650 50  0001 C CNN
@@
 $EndComp
 $Comp
-L power:+2V8 #PWR036
+L power:+2V8 #PWR040
 U 1 1 5BBBFBE8
 P 2700 3950
-F 0 "#PWR036" H 2700 3800 50  0001 C CNN
+F 0 "#PWR040" H 2700 3800 50  0001 C CNN
 F 1 "+2V8" V 2715 4078 50  0000 L CNN
 F 2 "" H 2700 3950 50  0001 C CNN
@@
 $EndComp
 $Comp
-L Device:R R10
+L Device:R R12
 U 1 1 5BBBFC54
 P 2200 3450
-F 0 "R10" H 2270 3496 50  0000 L CNN
+F 0 "R12" H 2270 3496 50  0000 L CNN
 F 1 "R" H 2270 3405 50  0000 L CNN
 F 2 "" V 2130 3450 50  0001 C CNN
@@
 $EndComp
 $Comp
-L Device:R R11
+L Device:R R13
 U 1 1 5BBBFCA5
 P 2450 3050
-F 0 "R11" H 2520 3096 50  0000 L CNN
+F 0 "R13" H 2520 3096 50  0000 L CNN
 F 1 "R" H 2520 3005 50  0000 L CNN
 F 2 "" V 2380 3050 50  0001 C CNN
@@
 	3400 3950 3400 3900
 $Comp
-L Device:R R12
+L Device:R R14
 U 1 1 5BBC053E
 P 3800 3350
-F 0 "R12" H 3870 3396 50  0000 L CNN
+F 0 "R14" H 3870 3396 50  0000 L CNN
 F 1 "R" H 3870 3305 50  0000 L CNN
 F 2 "" V 3730 3350 50  0001 C CNN
@@
 $EndComp
 $Comp
-L Device:R R13
+L Device:R R15
 U 1 1 5BBC057D
 P 4050 3750
-F 0 "R13" H 4120 3796 50  0000 L CNN
+F 0 "R15" H 4120 3796 50  0000 L CNN
 F 1 "R" H 4120 3705 50  0000 L CNN
 F 2 "" V 3980 3750 50  0001 C CNN

Commit message: Fixed shift register voltage translation
Parts:
- renumbered Q2 to Q1, Q3 to Q2, R12 to R10, R13 to R11, R14 to R12, R15 to R13
Changed lines of the file:
@@
 $Descr A4 11693 8268
 encoding utf-8
-Sheet 4 16
+Sheet 4 19
 Title ""
 Date ""
@@
 $EndDescr
 $Comp
-L Transistor_FET:BSS138 Q2
+L Transistor_FET:BSS138 Q1
 U 1 1 5BBBF528
 P 2850 3300
-F 0 "Q2" V 3193 3300 50  0000 C CNN
+F 0 "Q1" V 3193 3300 50  0000 C CNN
 F 1 "BSS138" V 3102 3300 50  0000 C CNN
 F 2 "Package_TO_SOT_SMD:SOT-23" H 3050 3225 50  0001 L CIN
@@
 I2C_STM32_SDA
 $Comp
-L Transistor_FET:BSS138 Q3
+L Transistor_FET:BSS138 Q2
 U 1 1 5BBBF64A
 P 3400 3700
-F 0 "Q3" V 3743 3700 50  0000 C CNN
+F 0 "Q2" V 3743 3700 50  0000 C CNN
 F 1 "BSS138" V 3652 3700 50  0000 C CNN
 F 2 "Package_TO_SOT_SMD:SOT-23" H 3600 3625 50  0001 L CIN
@@
 $EndComp
 $Comp
-L power:+3.3V #PWR039
+L power:+3.3V #PWR040
 U 1 1 5BBBF787
 P 2450 2650
-F 0 "#PWR039" H 2450 2500 50  0001 C CNN
+F 0 "#PWR040" H 2450 2500 50  0001 C CNN
 F 1 "+3.3V" H 2465 2823 50  0000 C CNN
 F 2 "" H 2450 2650 50  0001 C CNN
@@
 $EndComp
 $Comp
-L power:+2V8 #PWR040
+L power:+2V8 #PWR041
 U 1 1 5BBBFBE8
 P 2700 3950
-F 0 "#PWR040" H 2700 3800 50  0001 C CNN
+F 0 "#PWR041" H 2700 3800 50  0001 C CNN
 F 1 "+2V8" V 2715 4078 50  0000 L CNN
 F 2 "" H 2700 3950 50  0001 C CNN
@@
 $EndComp
 $Comp
-L Device:R R12
+L Device:R R10
 U 1 1 5BBBFC54
 P 2200 3450
-F 0 "R12" H 2270 3496 50  0000 L CNN
+F 0 "R10" H 2270 3496 50  0000 L CNN
 F 1 "R" H 2270 3405 50  0000 L CNN
 F 2 "" V 2130 3450 50  0001 C CNN
@@
 $EndComp
 $Comp
-L Device:R R13
+L Device:R R11
 U 1 1 5BBBFCA5
 P 2450 3050
-F 0 "R13" H 2520 3096 50  0000 L CNN
+F 0 "R11" H 2520 3096 50  0000 L CNN
 F 1 "R" H 2520 3005 50  0000 L CNN
 F 2 "" V 2380 3050 50  0001 C CNN
@@
 	3400 3950 3400 3900
 $Comp
-L Device:R R14
+L Device:R R12
 U 1 1 5BBC053E
 P 3800 3350
-F 0 "R14" H 3870 3396 50  0000 L CNN
+F 0 "R12" H 3870 3396 50  0000 L CNN
 F 1 "R" H 3870 3305 50  0000 L CNN
 F 2 "" V 3730 3350 50  0001 C CNN
@@
 $EndComp
 $Comp
-L Device:R R15
+L Device:R R13
 U 1 1 5BBC057D
 P 4050 3750
-F 0 "R15" H 4120 3796 50  0000 L CNN
+F 0 "R13" H 4120 3796 50  0000 L CNN
 F 1 "R" H 4120 3705 50  0000 L CNN
 F 2 "" V 3980 3750 50  0001 C CNN

Commit message: Added IC for level translation with ultrasonic sensors
Parts:
- R10: renamed from R11; footprint (none) -> Resistor_SMD:R_0805_2012Metric_Pad1.15x1.40mm_HandSolder
- R11: renamed from R12; footprint (none) -> Resistor_SMD:R_0805_2012Metric_Pad1.15x1.40mm_HandSolder
- R12: renamed from R13; footprint (none) -> Resistor_SMD:R_0805_2012Metric_Pad1.15x1.40mm_HandSolder
- R9: renamed from R10; footprint (none) -> Resistor_SMD:R_0805_2012Metric_Pad1.15x1.40mm_HandSolder
Changed lines of the file:
@@
 $Descr A4 11693 8268
 encoding utf-8
-Sheet 4 19
+Sheet 3 19
 Title ""
 Date ""
@@
 $EndComp
 $Comp
-L power:+3.3V #PWR040
+L power:+3.3V #PWR030
 U 1 1 5BBBF787
 P 2450 2650
-F 0 "#PWR040" H 2450 2500 50  0001 C CNN
+F 0 "#PWR030" H 2450 2500 50  0001 C CNN
 F 1 "+3.3V" H 2465 2823 50  0000 C CNN
 F 2 "" H 2450 2650 50  0001 C CNN
@@
 $EndComp
 $Comp
-L power:+2V8 #PWR041
+L power:+2V8 #PWR031
 U 1 1 5BBBFBE8
 P 2700 3950
-F 0 "#PWR041" H 2700 3800 50  0001 C CNN
+F 0 "#PWR031" H 2700 3800 50  0001 C CNN
 F 1 "+2V8" V 2715 4078 50  0000 L CNN
 F 2 "" H 2700 3950 50  0001 C CNN
@@
 $EndComp
 $Comp
-L Device:R R10
+L Device:R R9
 U 1 1 5BBBFC54
 P 2200 3450
-F 0 "R10" H 2270 3496 50  0000 L CNN
+F 0 "R9" H 2270 3496 50  0000 L CNN
 F 1 "R" H 2270 3405 50  0000 L CNN
-F 2 "" V 2130 3450 50  0001 C CNN
+F 2 "Resistor_SMD:R_0805_2012Metric_Pad1.15x1.40mm_HandSolder" V 2130 3450 50  0001 C CNN
 F 3 "~" H 2200 3450 50  0001 C CNN
 	1    2200 3450
@@
 $EndComp
 $Comp
-L Device:R R11
+L Device:R R10
 U 1 1 5BBBFCA5
 P 2450 3050
-F 0 "R11" H 2520 3096 50  0000 L CNN
+F 0 "R10" H 2520 3096 50  0000 L CNN
 F 1 "R" H 2520 3005 50  0000 L CNN
-F 2 "" V 2380 3050 50  0001 C CNN
+F 2 "Resistor_SMD:R_0805_2012Metric_Pad1.15x1.40mm_HandSolder" V 2380 3050 50  0001 C CNN
 F 3 "~" H 2450 3050 50  0001 C CNN
 	1    2450 3050
@@
 	3400 3950 3400 3900
 $Comp
-L Device:R R12
+L Device:R R11
 U 1 1 5BBC053E
 P 3800 3350
-F 0 "R12" H 3870 3396 50  0000 L CNN
+F 0 "R11" H 3870 3396 50  0000 L CNN
 F 1 "R" H 3870 3305 50  0000 L CNN
-F 2 "" V 3730 3350 50  0001 C CNN
+F 2 "Resistor_SMD:R_0805_2012Metric_Pad1.15x1.40mm_HandSolder" V 3730 3350 50  0001 C CNN
 F 3 "~" H 3800 3350 50  0001 C CNN
 	1    3800 3350
@@
 $EndComp
 $Comp
-L Device:R R13
+L Device:R R12
 U 1 1 5BBC057D
 P 4050 3750
-F 0 "R13" H 4120 3796 50  0000 L CNN
+F 0 "R12" H 4120 3796 50  0000 L CNN
 F 1 "R" H 4120 3705 50  0000 L CNN
-F 2 "" V 3980 3750 50  0001 C CNN
+F 2 "Resistor_SMD:R_0805_2012Metric_Pad1.15x1.40mm_HandSolder" V 3980 3750 50  0001 C CNN
 F 3 "~" H 4050 3750 50  0001 C CNN
 	1    4050 3750

Commit message: Footprint association
Parts:
- Q1, Q2: footprint Package_TO_SOT_SMD:SOT-23 -> Package_TO_SOT_SMD:SOT-23_Handsoldering
Changed lines of the file:
@@
 F 0 "Q1" V 3193 3300 50  0000 C CNN
 F 1 "BSS138" V 3102 3300 50  0000 C CNN
-F 2 "Package_TO_SOT_SMD:SOT-23" H 3050 3225 50  0001 L CIN
+F 2 "Package_TO_SOT_SMD:SOT-23_Handsoldering" H 3050 3225 50  0001 L CIN
 F 3 "https://www.fairchildsemi.com/datasheets/BS/BSS138.pdf" H 2850 3300 50  0001 L CNN
 	1    2850 3300
@@
 F 0 "Q2" V 3743 3700 50  0000 C CNN
 F 1 "BSS138" V 3652 3700 50  0000 C CNN
-F 2 "Package_TO_SOT_SMD:SOT-23" H 3600 3625 50  0001 L CIN
+F 2 "Package_TO_SOT_SMD:SOT-23_Handsoldering" H 3600 3625 50  0001 L CIN
 F 3 "https://www.fairchildsemi.com/datasheets/BS/BSS138.pdf" H 3400 3700 50  0001 L CNN
 	1    3400 3700
