File: I2C.sch (KiCad schematic (older format))
At the start: 7 parts, among them U9 TCA9517DR

Commit message: Update PCB
Parts:
- C20, C21: footprint (none) -> Capacitor_SMD:C_0805_2012Metric_Pad1.15x1.40mm_HandSolder
- R10, R11, R2, R9: footprint (none) -> Resistor_SMD:R_0805_2012Metric_Pad1.15x1.40mm_HandSolder
- U9: footprint Package_SO:SOIC-8_3.9x4.9mm_P1.27mm -> Package_SO:TSSOP-8_3x3mm_P0.65mm
Changed lines of the file:
@@
 F 0 "U9" H 3200 2711 50  0000 C CNN
 F 1 "TCA9517DR" H 3200 2620 50  0000 C CNN
-F 2 "Package_SO:SOIC-8_3.9x4.9mm_P1.27mm" H 2800 3650 50  0001 C CNN
+F 2 "Package_SO:TSSOP-8_3x3mm_P0.65mm" H 2800 3650 50  0001 C CNN
 F 3 "https://www.ti.com/lit/ds/symlink/tca9517.pdf" H 2900 3750 50  0001 C CNN
 	1    3200 3300
@@
 F 0 "R2" H 2370 3046 50  0000 L CNN
 F 1 "10k" H 2370 2955 50  0000 L CNN
-F 2 "" V 2230 3000 50  0001 C CNN
+F 2 "Resistor_SMD:R_0805_2012Metric_Pad1.15x1.40mm_HandSolder" V 2230 3000 50  0001 C CNN
 F 3 "~" H 2300 3000 50  0001 C CNN
 	1    2300 3000
@@
 F 0 "R9" H 2670 3046 50  0000 L CNN
 F 1 "10k" H 2670 2955 50  0000 L CNN
-F 2 "" V 2530 3000 50  0001 C CNN
+F 2 "Resistor_SMD:R_0805_2012Metric_Pad1.15x1.40mm_HandSolder" V 2530 3000 50  0001 C CNN
 F 3 "~" H 2600 3000 50  0001 C CNN
 	1    2600 3000
@@
 F 0 "R10" H 4020 2996 50  0000 L CNN
 F 1 "10k" H 4020 2905 50  0000 L CNN
-F 2 "" V 3880 2950 50  0001 C CNN
+F 2 "Resistor_SMD:R_0805_2012Metric_Pad1.15x1.40mm_HandSolder" V 3880 2950 50  0001 C CNN
 F 3 "~" H 3950 2950 50  0001 C CNN
 	1    3950 2950
@@
 F 0 "R11" H 4320 2996 50  0000 L CNN
 F 1 "10k" H 4320 2905 50  0000 L CNN
-F 2 "" V 4180 2950 50  0001 C CNN
+F 2 "Resistor_SMD:R_0805_2012Metric_Pad1.15x1.40mm_HandSolder" V 4180 2950 50  0001 C CNN
 F 3 "~" H 4250 2950 50  0001 C CNN
 	1    4250 2950
@@
 F 0 "C20" H 2965 2446 50  0000 L CNN
 F 1 "100n" H 2965 2355 50  0000 L CNN
-F 2 "" H 2888 2250 50  0001 C CNN
+F 2 "Capacitor_SMD:C_0805_2012Metric_Pad1.15x1.40mm_HandSolder" H 2888 2250 50  0001 C CNN
 F 3 "~" H 2850 2400 50  0001 C CNN
 	1    2850 2400
@@
 F 0 "C21" H 3715 2446 50  0000 L CNN
 F 1 "100n" H 3715 2355 50  0000 L CNN
-F 2 "" H 3638 2250 50  0001 C CNN
+F 2 "Capacitor_SMD:C_0805_2012Metric_Pad1.15x1.40mm_HandSolder" H 3638 2250 50  0001 C CNN
 F 3 "~" H 3600 2400 50  0001 C CNN
 	1    3600 2400

Commit message: Updated I2C schematic comments and IOC for clock configuration
Other:
- note added: "Essayer 1k en cas de problème\nRester en dessous de 6 mA."
Changed lines of the file:
@@
 Wire Wire Line
 	3600 2600 3950 2600
+Wire Notes Line
+	3800 2750 4500 2750
+Wire Notes Line
+	4500 2750 4500 3150
+Wire Notes Line
+	4500 3150 3800 3150
+Wire Notes Line
+	3800 3150 3800 2750
+Text Notes 4550 3000 0    50   ~ 0
+Essayer 1k en cas de problème\nRester en dessous de 6 mA.
 $EndSCHEMATC
