File: ultraphotonicsense-elec.kicad_pcb (KiCad board)
At the start: 2 copper layers, 83 x 38 mm, 79 parts, among them J1 Conn_Debug, J10 Conn_01x04, J11 Conn_01x04, J12 Conn_01x04, J13 Conn_01x04, J2 Conn_01x05, J3 Conn_01x05, J4 Conn_01x05, J5 Conn_01x05, J6 Conn_01x05, J7 Conn_01x05, J8 Conn_01x05, J9 Conn_01x05, P1 CAN_conn, P2 CAN_conn, Q1 BSS138, Q2 BSS138, Q3 BSS138, Q4 BSS138, Q5 BSS138, U1 TXB0108PW, U2 74HC164, U3 TCAN332, U4 LD1117S50TR_SOT223, U5 LD1117S33TR_SOT223, U6 LP38693MP-ADJ, U7 STM32F303K8Tx, Y1 Crystal

Commit message: cleanup
Routing:
- net /Level_Conv_0/IN_3V3: track 33.5 -> 28.5 mm
- net /Level_Conv_2/IN_3V3: track 110.7 -> 107.7 mm
Changed lines of the file:
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@@
     (thickness 1.6)
     (drawings 32)
-    (tracks 725)
+    (tracks 721)
     (zones 0)
     (modules 79)
@@
   (segment (start 83.85 69.55) (end 84.275 69.125) (width 0.25) (layer B.Cu) (net 45))
   (segment (start 83.85 71.125) (end 83.85 69.55) (width 0.25) (layer B.Cu) (net 45) (status 10))
-  (segment (start 84.925 69.125) (end 85.771032 69.125) (width 0.25) (layer B.Cu) (net 45) (status 10))
-  (segment (start 85.771032 69.125) (end 87.00001 70.353978) (width 0.25) (layer B.Cu) (net 45))
-  (segment (start 87.00001 70.353978) (end 87.00001 72.74999) (width 0.25) (layer B.Cu) (net 45))
   (segment (start 84.925 69.125) (end 83.75 69.125) (width 0.25) (layer B.Cu) (net 45) (status 10))
   (segment (start 83.75 69.125) (end 83.625 69.125) (width 0.25) (layer B.Cu) (net 45))
@@
   (segment (start 77.846022 73.32501) (end 68.75 73.32501) (width 0.25) (layer B.Cu) (net 60))
   (segment (start 68.75 73.32501) (end 67.29999 73.32501) (width 0.25) (layer B.Cu) (net 60))
-  (segment (start 51 71.75) (end 47.95 71.75) (width 0.25) (layer B.Cu) (net 60))
   (segment (start 56.25 47.125) (end 56.25 47) (width 0.25) (layer B.Cu) (net 60) (status 30))
   (segment (start 51 71.75) (end 48.35 71.75) (width 0.25) (layer B.Cu) (net 60))

Commit message: small fixes
Routing:
- net GND: track 378.5 -> 437.1 mm
- net +2V8: track 165.8 -> 151.6 mm
- net /STM32F303K8/I2C_SCL: track 17.4 -> 16.9 mm

Commit message: Update PCB
Parts:
- removed Q1, Q2, Q3, Q4, Q5: BSS138, Package_TO_SOT_SMD:SOT-23_Handsoldering
- removed R17, R18, R19, R20: R, Resistor_SMD:R_0805_2012Metric_Pad1.15x1.40mm_HandSolder
- added C17: 100n, Capacitor_SMD:C_0805_2012Metric_Pad1.15x1.40mm_HandSolder, B.Cu at (76.6, 70.6)
- added C18: 100n, Capacitor_SMD:C_0805_2012Metric_Pad1.15x1.40mm_HandSolder, F.Cu at (91.2, 57.2)
- added C19: 100n, Capacitor_SMD:C_0805_2012Metric_Pad1.15x1.40mm_HandSolder, F.Cu at (93.6, 57.2)
- added C20: 100n, Capacitor_SMD:C_0805_2012Metric_Pad1.15x1.40mm_HandSolder, B.Cu at (85.0, 66.4)
- added C21: 100n, Capacitor_SMD:C_0805_2012Metric_Pad1.15x1.40mm_HandSolder, B.Cu at (83.0, 66.4)
- added R2: 10k, Resistor_SMD:R_0805_2012Metric_Pad1.15x1.40mm_HandSolder, B.Cu at (93.0, 68.2)
- added SW1: SW_SPST, PhenixRobotik:SW_SPST_CK_KSS_3.7x5.5mm, F.Cu at (77.7, 71.8)
- added U10: SN74AHC1G08DBV, Package_TO_SOT_SMD:SOT-23-5_HandSoldering, B.Cu at (71.8, 65.8)
- added U8: TXB0104PW, Package_SO:TSSOP-14_4.4x5mm_P0.65mm, B.Cu at (92.3, 57.5)
- added U9: TCA9517DR, Package_SO:TSSOP-8_3x3mm_P0.65mm, F.Cu at (83.9, 66.0)
- C10, C9: footprint Capacitor_SMD:C_0805_2012Metric_Pad1.15x1.40mm_HandSolder -> Capacitor_SMD:C_0603_1608Metric_Pad1.05x0.95mm_HandSolder
- D1: footprint Diode_SMD:D_2114_3652Metric_Castellated -> Diode_SMD:D_SMA
- R1, R13, R14: value R -> 10k
- R10, R11, R9: value R -> 10k; moved to B.Cu
- R12: value R -> 1k; moved to B.Cu
- R16: value 1k -> 330
- R3: value R -> 700
- R4: value R -> 500
- R5: value R -> 330
- R6: value R2 -> 6.8k
- R7: value R1 -> 9.1k
- R8: value R -> 280
- Y1: value Crystal -> 16MHz
- moved R14 28.3 mm to (66.3, 67.6), turned to 0 degrees
- moved R13 19.4 mm to (66.4, 65.6), turned to 0 degrees
- moved R9 15.3 mm to (93.0, 66.2), turned to 180 degrees
- moved JP2 9.71 mm to (84.2, 70.6)
- moved R12 7.64 mm to (78.8, 70.6)
- moved R11 6.26 mm to (79.8, 67.4), turned to 180 degrees
- moved R10 5.79 mm to (79.8, 65.4), turned to 180 degrees
- moved R15 4.57 mm to (81.8, 70.6), turned to 90 degrees
- moved U2 2.03 mm to (101.5, 57.5)
- moved Y1 1.50 mm to (80.4, 59.4)
- moved C9 0.65 mm to (82.4, 60.2)
- moved C10 0.65 mm to (82.4, 56.2)
- moved C11 0.32 mm to (77.2, 59.2)
- moved D1 0.25 mm to (42.0, 45.2)
Connections:
- net /Level_Conv_0/OUT_2V8 renamed Net-(U2-Pad1)
- C11 pad 2: /Level_Conv_2/IN_3V3 -> /NRST_Logic/NRST
- J1 pad 2: /Level_Conv_2/IN_3V3 -> /NRST_Logic/NRST_DBG
- P1 pad 2: /Level_Conv_2/IN_3V3 -> /Power_CAN/NRST
- P2 pad 2: /Level_Conv_2/IN_3V3 -> /Power_CAN/NRST
- R10 pad 2: /STM32F303K8/I2C_SCL -> /STM32F303K8/I2C_SDA
- R11 pad 1: ToF_SCL -> +3V3
- R11 pad 2: +2V8 -> /STM32F303K8/I2C_SCL
- R12 pad 1: ToF_SDA -> Net-(C17-Pad2)
- R12 pad 2: +2V8 -> /NRST_Logic/NRST_DBG
- R13 pad 1: /Level_Conv_2/IN_3V3 -> +3V3
- R13 pad 2: +3V3 -> /Power_CAN/NRST
- R14 pad 1: /Level_Conv_2/OUT_2V8 -> +3V3
- R14 pad 2: +2V8 -> Net-(C17-Pad2)
- R9 pad 1: +3V3 -> +2V8
- R9 pad 2: /STM32F303K8/I2C_SDA -> ToF_SDA
- U2 pad 8: /Level_Conv_1/OUT_2V8 -> Net-(U2-Pad8)
- U2 pad 9: /Level_Conv_2/OUT_2V8 -> Net-(U2-Pad9)
- U3 pad 5: Net-(U3-Pad5) -> (no net)
- U3 pad 8: Net-(U3-Pad8) -> (no net)
- U6 pad 1: /Level_Conv_2/IN_3V3 -> /Power_CAN/NRST
- U7 pad 15: Net-(U7-Pad15) -> /STM32F303K8/I2C_EN
- U7 pad 26: Net-(U7-Pad26) -> (no net)
- U7 pad 27: /Level_Conv_0/IN_3V3 -> /STM32F303K8/TOF_RESET_DATA
- U7 pad 28: /Level_Conv_1/IN_3V3 -> /STM32F303K8/TOF_RESET_SHIFT
- U7 pad 29: Net-(U7-Pad29) -> (no net)
- U7 pad 4: /Level_Conv_2/IN_3V3 -> /NRST_Logic/NRST
Routing:
- net /Level_Conv_2/IN_3V3: track 107.7 -> 0.00 mm, vias 4 -> 0
- net /Power_CAN/NRST: track 0.00 -> 61.4 mm, vias 0 -> 1
- net GND: track 437.1 -> 495.0 mm, vias 10 -> 14
- net +3V3: track 152.1 -> 184.1 mm, vias 8 -> 9
- net /NRST_Logic/NRST: track 0.00 -> 31.6 mm, vias 0 -> 3
- net /Level_Conv_0/IN_3V3: track 28.5 -> 0.00 mm, vias 1 -> 0
- net /STM32F303K8/TOF_RESET_DATA: track 0.00 -> 28.5 mm, vias 0 -> 1
- net /STM32F303K8/TOF_RESET_SHIFT: track 0.00 -> 27.6 mm, vias 0 -> 1
- net /Level_Conv_1/IN_3V3: track 27.2 -> 0.00 mm, vias 1 -> 0
- net Net-(U2-Pad1): track 39.1 -> 19.4 mm
- net /STM32F303K8/I2C_EN: track 0.00 -> 19.5 mm, vias 0 -> 2
- net Net-(C17-Pad2): track 0.00 -> 14.6 mm
- net /NRST_Logic/NRST_DBG: track 0.00 -> 14.0 mm, vias 0 -> 1
- net /Level_Conv_2/OUT_2V8: track 9.79 -> 0.00 mm
- net +2V8: track 151.6 -> 142.2 mm, vias 2 -> 5
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Other:
- board text added: "https://github.com /PhenixRobotik /ultraphotonicsense-elec"
- board text removed: "https://github.com/PhenixRobotik/ultraphotonicsense-elec"

Commit message: Update silkscreen
Parts:
- C18, C19: moved to B.Cu
- moved C18 2.73 mm to (90.2, 54.7), turned to 180 degrees
- moved C19 2.59 mm to (94.2, 54.7), turned to 0 degrees
- moved U8 1.06 mm to (92.2, 58.5)
Routing:
- net +3V3: track 184.1 -> 190.2 mm, vias 9 -> 8
- net GND: track 495.0 -> 500.5 mm, vias 14 -> 13
- net +2V8: track 142.2 -> 146.9 mm, vias 5 -> 4
- net Net-(U2-Pad1): track 19.4 -> 17.0 mm
- net Net-(U2-Pad8): track 3.48 -> 4.72 mm
- net Net-(U2-Pad9): track 5.10 -> 6.12 mm
