File: ultraphotonicsense-elec.sch (KiCad schematic (older format))
At the start: 19 parts, among them J1 Conn_Debug, SW1 SW_SPST, U1 TXB0108PW, U2 74HC164, U8 TXB0104PW

Commit message: Update PCB
Parts:
- removed C17: 100n, symbol Device:C
- removed SW1: SW_SPST, symbol Switch:SW_SPST
- C18, C19: footprint (none) -> Capacitor_SMD:C_0805_2012Metric_Pad1.15x1.40mm_HandSolder
Connections:
- wire segments 137 -> 129
Changed lines of the file:
@@
 F0 "NRST_Logic" 50
 F1 "nrst_logic.sch" 50
-F2 "NRST_1" I L 2600 3850 50
-F3 "NRST_2" I L 2600 3950 50
-F4 "NRST" O R 3300 3900 50
+F2 "NRST" O R 3300 3900 50
+F3 "NRST_DBG" I L 2600 3850 50
+F4 "NRST_CAN" I L 2600 3950 50
 $EndSheet
 Wire Wire Line
@@
 Wire Wire Line
 	2450 3750 2450 3850
-Wire Wire Line
-	2450 3850 2600 3850
 Wire Wire Line
 	1150 4450 1450 4450
@@
 	2450 4200 2450 3950
 Wire Wire Line
-	2450 3950 2600 3950
-Wire Wire Line
 	2200 4400 2500 4400
 Wire Wire Line
@@
 Wire Wire Line
 	1350 5250 1450 5250
-$Comp
-L Switch:SW_SPST SW1
-U 1 1 5F7EFC79
-P 2700 2350
-F 0 "SW1" H 2700 2585 50  0000 C CNN
-F 1 "SW_SPST" H 2700 2494 50  0000 C CNN
-F 2 "" H 2700 2350 50  0001 C CNN
-F 3 "~" H 2700 2350 50  0001 C CNN
-	1    2700 2350
-	1    0    0    -1
-$EndComp
-$Comp
-L Device:C C17
-U 1 1 5F7F11AE
-P 2700 2650
-F 0 "C17" V 2448 2650 50  0000 C CNN
-F 1 "100n" V 2539 2650 50  0000 C CNN
-F 2 "" H 2738 2500 50  0001 C CNN
-F 3 "~" H 2700 2650 50  0001 C CNN
-	1    2700 2650
-	0    1    1    0
-$EndComp
-$Comp
-L power:GND #PWR017
-U 1 1 5F7F1B41
-P 2950 2700
-F 0 "#PWR017" H 2950 2450 50  0001 C CNN
-F 1 "GND" H 2955 2527 50  0000 C CNN
-F 2 "" H 2950 2700 50  0001 C CNN
-F 3 "" H 2950 2700 50  0001 C CNN
-	1    2950 2700
-	1    0    0    -1
-$EndComp
-Wire Wire Line
-	2950 2350 2950 2650
-Connection ~ 2450 3750
-Wire Wire Line
-	2450 2350 2450 2650
-Wire Wire Line
-	2450 2650 2550 2650
-Connection ~ 2450 2650
-Wire Wire Line
-	2450 2650 2450 3750
-Wire Wire Line
-	2850 2650 2950 2650
-Connection ~ 2950 2650
-Wire Wire Line
-	2450 2350 2500 2350
-Wire Wire Line
-	2900 2350 2950 2350
-Wire Wire Line
-	2950 2650 2950 2700
 $Sheet
 S 3550 3050 1300 1750
@@
 F 0 "C18" H 5465 4896 50  0000 L CNN
 F 1 "100n" H 5465 4805 50  0000 L CNN
-F 2 "" H 5388 4700 50  0001 C CNN
+F 2 "Capacitor_SMD:C_0805_2012Metric_Pad1.15x1.40mm_HandSolder" H 5388 4700 50  0001 C CNN
 F 3 "~" H 5350 4850 50  0001 C CNN
 	1    5350 4850
@@
 F 0 "C19" H 6415 4896 50  0000 L CNN
 F 1 "100n" H 6415 4805 50  0000 L CNN
-F 2 "" H 6338 4700 50  0001 C CNN
+F 2 "Capacitor_SMD:C_0805_2012Metric_Pad1.15x1.40mm_HandSolder" H 6338 4700 50  0001 C CNN
 F 3 "~" H 6300 4850 50  0001 C CNN
 	1    6300 4850
@@
 	6300 5000 6300 5050
 Connection ~ 6300 5050
+Wire Wire Line
+	2450 3850 2600 3850
+Wire Wire Line
+	2450 3950 2600 3950
 $EndSCHEMATC

Commit message: Added optional pull-up on UART TX
Parts:
- added R?: DNE, symbol Device:R
Connections:
- wire segments 129 -> 132
Changed lines of the file:
@@
 	3300 3900 3450 3900
 Wire Wire Line
-	2300 3150 3550 3150
+	2300 3150 2950 3150
 Wire Wire Line
 	2300 3250 3550 3250
@@
 Wire Wire Line
 	2450 3950 2600 3950
+$Comp
+L Device:R R?
+U 1 1 5F8BB2B7
+P 2950 2900
+F 0 "R?" H 3020 2946 50  0000 L CNN
+F 1 "DNE" H 3020 2855 50  0000 L CNN
+F 2 "" V 2880 2900 50  0001 C CNN
+F 3 "~" H 2950 2900 50  0001 C CNN
+	1    2950 2900
+	1    0    0    -1
+$EndComp
+$Comp
+L power:+3V3 #PWR?
+U 1 1 5F8BB82E
+P 2950 2650
+F 0 "#PWR?" H 2950 2500 50  0001 C CNN
+F 1 "+3V3" H 2965 2823 50  0000 C CNN
+F 2 "" H 2950 2650 50  0001 C CNN
+F 3 "" H 2950 2650 50  0001 C CNN
+	1    2950 2650
+	1    0    0    -1
+$EndComp
+Wire Wire Line
+	2950 2650 2950 2750
+Wire Wire Line
+	2950 3050 2950 3150
+Connection ~ 2950 3150
+Wire Wire Line
+	2950 3150 3550 3150
 $EndSCHEMATC
